File: dc01.kicad_sch (KiCad schematic)
At the start: 76 parts, among them J1 USB_C_Receptacle_USB2.0, J2 PROG/DEBUG, J3 Conn_01x06, J4 RJ12, J5 RJ12, J6 Screw_Terminal_01x02, J7 Screw_Terminal_01x02, J8 Conn_01x02, U1 STM32F103C8Tx, U2 AMS1117-3.3, U3 ADM2483xRW, U4 ADUM1250, U6 LM78M05_TO252, U7 INA219AxDCN, Y1 8 MHz

Commit message: Remove unused parts.
Parts:
- removed C10, C11, C12, C13, C16: 100n, Capacitor_SMD:C_0805_2012Metric, symbol Device:C
- removed C14: 22u, Capacitor_SMD:C_0805_2012Metric, symbol Device:C
- removed C15: 22u/25V, Capacitor_SMD:C_0805_2012Metric, symbol Device:C
- removed C17: 470p, Capacitor_THT:C_Disc_D12.5mm_W5.0mm_P10.00mm, symbol Device:C
- removed D5: 1N4007, Diode_SMD:D_SOD-123, symbol Device:D
- removed D6: LED-BLUE, LED_SMD:LED_0805_2012Metric, symbol Device:LED
- removed D8: SM712_SOT23, Package_TO_SOT_SMD:SOT-23, symbol Diode:SM712_SOT23
- removed J6, J7: Screw_Terminal_01x02, TerminalBlock_4Ucon:TerminalBlock_4Ucon_1x02_P3.50mm_Horizontal, symbol Connector:Screw_Terminal_01x02
- removed JP5, JP6: SJ_2_Open, Jumper:SolderJumper-2_P1.3mm_Open_RoundedPad1.0x1.5mm, symbol Jumper:SolderJumper_2_Open
- removed JP7: SJ3_Bridged12, Jumper:SolderJumper-3_P1.3mm_Bridged12_RoundedPad1.0x1.5mm_NumberLabels, symbol Jumper:SolderJumper_3_Bridged12
- removed PS1: AM2D-0505SZ, Converter_DCDC:Converter_DCDC_XP_POWER-IHxxxxS_THT, symbol Converter_DCDC:IH0505S
- removed R10: 1k, Resistor_SMD:R_0805_2012Metric, symbol Device:R
- removed R11: 0.1R, Resistor_SMD:R_1206_3216Metric, symbol Device:R
- removed R12, R13, R14, R16, R8, R9: 10k, Resistor_SMD:R_0805_2012Metric, symbol Device:R
- removed R15: 220R, Resistor_SMD:R_0805_2012Metric, symbol Device:R
- removed R18: 10M, Resistor_THT:R_Axial_DIN0207_L6.3mm_D2.5mm_P10.16mm_Horizontal, symbol Device:R
- removed TP1, TP2, TP3, TP4, TP5: TestPoint, TestPoint:TestPoint_Pad_D1.0mm, symbol Connector:TestPoint
- removed TP7: TestPoint, TestPoint:TestPoint_Loop_D3.50mm_Drill1.4mm_Beaded, symbol Connector:TestPoint
- removed U3: ADM2483xRW, Package_SO:SOIC-16W_7.5x10.3mm_P1.27mm, symbol Interface_UART:ADM2483xRW
- removed U4: ADUM1250, Package_SO:SO-8_3.9x4.9mm_P1.27mm, symbol Interface_I2C:ADUM1250
- removed U6: LM78M05_TO252, Package_TO_SOT_SMD:TO-252-2, symbol Regulator_Linear:LM78M05_TO252
- removed U7: INA219AxDCN, Package_TO_SOT_SMD:SOT-23-8, symbol Analog_ADC:INA219AxDCN
Connections:
- removed net +12VA: J4.1, J4.6, J5.1, J5.6
- removed net GNDA: J4.2, J4.5, J5.2, J5.5
- net I2C_SCL: no longer names the net of U1.45 (PB8)
- net I2C_SDA: no longer names the net of U1.46 (PB9)
- net MTB-BUS+: no longer names the net of J5.3
- net MTB-BUS+: no longer J4.3
- net MTB-BUS-: no longer names the net of J5.4
- net MTB-BUS-: no longer J4.4
- net USART_MTB_DIR: no longer names the net of U1.20 (PB2)
- net USART_MTB_RX: no longer names the net of U1.22 (PB11)
- net USART_MTB_TX: no longer names the net of U1.21 (PB10)
Other:
- note removed: "1 kV for 10 s"
- note removed: "250 mA max (bus shorted)"
- note removed: "CC10K-470"
- note removed: "Either PS1 is fitted or external power supply on J6 should be provided. Exactly one of JP5 & JP6 should be closed."
- note removed: "VR37000001005JA100"
- note removed: "optional"
- title: MTB-USB v4 -> DCC cutter DC-01

Commit message: Add & wire relay part.
Parts:
- added C10, C11: 22u, Capacitor_SMD:C_0805_2012Metric, symbol Device:C
- added D10, D6: GR, symbol Device:LED
- added D11, D5: 1N4148, Diode_THT:D_DO-35_SOD27_P7.62mm_Horizontal, symbol Diode:1N4148
- added D8, D9: YEL, symbol Device:LED
- added F1, F2: 1A, symbol Device:Polyfuse
- added J6, J7: Conn_01x02, symbol Connector_Generic:Conn_01x02
- added K1, K2: AZ850-5, Relay_THT:Relay_DPDT_FRT5, symbol Relay:AZ850-x
- added Q1, Q2: 2N7002, Package_TO_SOT_SMD:SOT-23, symbol Transistor_FET:2N7002
- added R10, R11, R12, R9: 1k, symbol Device:R
- added R13, R8: 10k, Resistor_SMD:R_0805_2012Metric_Pad1.20x1.40mm_HandSolder, symbol Device:R
Connections:
- net +5V: now also C10.1, C11.1, D11.1 (K), D5.1 (K), K1.1, K2.1
- net GND: now also C10.2, C11.2, Q1.2 (S), Q2.2 (S), R13.2, R8.2
- net J2: now reaches J5.1
- net J2: now also D10.2 (A), D9.1 (K), F1.2, J7.1 (Pin_1)
- net TW2: now reaches J5.2
- net TW2: now also J4.2
- net TW3: now reaches J5.3
- net TW3: now also J4.3
- net TW4: now reaches J5.4
- net TW4: now also J4.4
- net TW5: now reaches J5.5
- net TW5: now also J4.5
- net K2: now reaches J5.6
- net K2: now also F2.2, J7.2 (Pin_2), R11.2, R12.1
- net J1: now reaches J4.1
- net J1: now also D6.2 (A), D8.1 (K), J6.1 (Pin_1), K1.7
- net K1: now reaches J4.6
- net K1: now also J6.2 (Pin_2), K2.7, R10.2, R9.1
- net REL1CTRL: now reaches U1.18 (PB0)
- net REL1CTRL: now also Q1.1 (G), R8.1
- net REL1TESTIN1: now reaches U1.19 (PB1)
- net REL1TESTIN1: now also K1.4
- net REL1TESTIN2: now reaches U1.20 (PB2)
- net REL1TESTIN2: now also K1.2
- net REL1TESTOUT: now reaches U1.39 (PB3)
- net REL1TESTOUT: now also K1.3
- net REL2CTRL: now reaches U1.40 (PB4)
- net REL2CTRL: now also Q2.1 (G), R13.1
- net REL2TESTIN1: now reaches U1.41 (PB5)
- net REL2TESTIN1: now also K2.4
- net REL2TESTIN2: now reaches U1.42 (PB6)
- net REL2TESTIN2: now also K2.2
- net REL2TESTOUT: now reaches U1.43 (PB7)
- net REL2TESTOUT: now also K2.3
- new net: D9.2 (A), R11.1
- new net: D8.2 (A), R10.1
- new net: D5.2 (A), K1.10, Q1.3 (D)
- new net: F1.1, K1.8
- new net: D10.1 (K), R12.2
- new net: D6.1 (K), R9.2
- new net: F2.1, K2.8
- new net: D11.2 (A), K2.10, Q2.3 (D)
- no-connect marks 28 -> 27
Other:
- moved on the sheet: C8, C9, D1, D2, D3, D4, J2, J3, J4, J5, JP1, JP2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

Commit message: Add relay-power indication LEDs.
Parts:
- added D12, D13: BLUE, symbol Device:LED
- added R14, R15: 1k, symbol Device:R
Connections:
- net GND: now also R14.2, R15.2
- net REL1CTRL: now also D12.2 (A)
- net REL2CTRL: now also D13.2 (A)
- new net: D13.1 (K), R15.1
- new net: D12.1 (K), R14.1
Other:
- moved on the sheet: C10, C11, D10, D11, D5, D6, D8, D9, F1, F2, J4, J5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

Commit message: Add buttons.
Parts:
- added R16, R18: 10k, symbol Device:R
- added SW1, SW2: SW_Push, symbol Switch:SW_Push
- C8: value 22u -> 10u
Connections:
- net +3V3: now also R16.2, R18.2
- net GND: now also SW1.1, SW2.1
- net SW1: now reaches U1.21 (PB10)
- net SW1: now also R16.1, SW1.2
- net SW2: now reaches U1.22 (PB11)
- net SW2: now also R18.1, SW2.2
- no-connect marks 27 -> 25
Other:
- moved on the sheet: D1, D2, D3, D4, R3, R5, R6, R7, TP6

Commit message: Add override switch.
Parts:
- added R19: 10k, symbol Device:R
- added SW3: SW_Push, symbol Switch:SW_Push
Connections:
- net +3V3: now also R19.2
- net GND: now also SW3.1
- net SW_OVERRIDE: now reaches U1.46 (PB9)
- net SW_OVERRIDE: now also R19.1, SW3.2
- net SW1 renamed SW_GO
- net SW2 renamed SW_STOP
- no-connect marks 25 -> 24
Other:
- moved on the sheet: R16, R18, SW2

Commit message: Add parts, several minor enhancements.
Parts:
- removed SW3: SW_Push, symbol Switch:SW_Push
- added D?: YEL, LED_SMD:LED_0805_2012Metric, symbol Device:LED
- added D?: RED, LED_SMD:LED_0805_2012Metric, symbol Device:LED
- added D?: GR, LED_SMD:LED_0805_2012Metric, symbol Device:LED
- added R? (x3): 1k, Resistor_SMD:R_0805_2012Metric, symbol Device:R
- added SW?: MFP 113 D, Button_Switch_THT:SW_Slide_1P2T_CK_OS102011MS2Q, symbol Switch:SW_SPDT
- D1: value LED-GR -> GR
- D10, D12, D13, D6, D8, D9: footprint (none) -> LED_SMD:LED_0805_2012Metric
- D2: value LED-YEL -> YEL
- D3: value LED-RED -> RED
- D4: value LED-BLUE -> BLUE
- F1, F2: footprint (none) -> Fuse:Fuse_1206_3216Metric
- R10, R11, R12, R14, R15, R16, R18, R19, R9: footprint (none) -> Resistor_SMD:R_0805_2012Metric
- SW1, SW2: footprint (none) -> Button_Switch_THT:SW_PUSH_6mm_H4.3mm
Connections:
- net +3V3: now also R?.2
- net GND: now also D?.1 (K), D?.1 (K), SW?.2 (B)
- net SW_GO: now also U1.14 (PA4); no longer U1.21 (PB10)
- net SW_OVERRIDE: now also U1.16 (PA6), D?.1 (K), SW?.3 (C); no longer U1.46 (PB9)
- net SW_STOP: now also U1.15 (PA5); no longer U1.22 (PB11)
- new net: D?.2 (A), R?.1 (x3)
- new net LED_GO: R?.2, U1.21 (PB10)
- new net LED_STOP: R?.2, U1.22 (PB11)
- no-connect marks 24 -> 23
Other:
- note added: "JLCPCB tooling holes"
- note added: "USB specification allows max 10u"
- moved on the sheet: C11, D1, D10, D2, D3, D4, D7, D9, F1, F2, H1, H2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

Commit message: Add outputs.
Parts:
- added J10, J9: Conn_01x02, symbol Connector_Generic:Conn_01x02
- added R23, R24: 470R, symbol Device:R
- added U3, U4: PC817, Package_DIP:DIP-4_W7.62mm, symbol Isolator:PC817
- gave numbers to parts that had none: 7
Connections:
- net GND: now also U3.2, U4.2
- net OUT_ALERT: now reaches U1.45 (PB8)
- net OUT_ALERT: now also R23.1
- net OUT_ON: now reaches U1.46 (PB9)
- net OUT_ON: now also R24.1
- new net: J9.1 (Pin_1), U3.4
- new net: J9.2 (Pin_2), U3.3
- new net: R24.2, U4.1
- new net: J10.1 (Pin_1), U4.4
- new net: J10.2 (Pin_2), U4.3
- new net: R23.2, U3.1
- no-connect marks 23 -> 21
Other:
- moved on the sheet: C8, C9, H1, H2, H3, J3, JP2, JP3, R4, U2

Commit message: Add footprints.
Parts:
- J10, J6, J7, J9: footprint (none) -> TerminalBlock_Euroclamp:MVE252-5-V
- R23, R24: footprint (none) -> Resistor_SMD:R_0805_2012Metric
Changed lines of the file:
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@@
       (effects (font (size 1.27 1.27)) (justify left))
     )
-    (property "Footprint" "" (id 2) (at 175.26 143.51 0)
+    (property "Footprint" "TerminalBlock_Euroclamp:MVE252-5-V" (id 2) (at 175.26 143.51 0)
       (effects (font (size 1.27 1.27)) hide)
     )
@@
     (property "Reference" "R24" (id 0) (at 140.97 152.7642 90))
     (property "Value" "470R" (id 1) (at 140.97 155.3011 90))
-    (property "Footprint" "" (id 2) (at 140.97 159.258 90)
+    (property "Footprint" "Resistor_SMD:R_0805_2012Metric" (id 2) (at 140.97 159.258 90)
       (effects (font (size 1.27 1.27)) hide)
     )
@@
       (effects (font (size 1.27 1.27)) (justify left))
     )
-    (property "Footprint" "" (id 2) (at 175.26 157.48 0)
+    (property "Footprint" "TerminalBlock_Euroclamp:MVE252-5-V" (id 2) (at 175.26 157.48 0)
       (effects (font (size 1.27 1.27)) hide)
     )
@@
     (property "Reference" "J6" (id 0) (at 180.34 97.9002 0))
     (property "Value" "Conn_01x02" (id 1) (at 180.34 100.4371 0))
-    (property "Footprint" "" (id 2) (at 180.34 102.87 0)
+    (property "Footprint" "TerminalBlock_Euroclamp:MVE252-5-V" (id 2) (at 180.34 102.87 0)
       (effects (font (size 1.27 1.27)) hide)
     )
@@
     (property "Reference" "R23" (id 0) (at 140.97 138.7942 90))
     (property "Value" "470R" (id 1) (at 140.97 141.3311 90))
-    (property "Footprint" "" (id 2) (at 140.97 145.288 90)
+    (property "Footprint" "Resistor_SMD:R_0805_2012Metric" (id 2) (at 140.97 145.288 90)
       (effects (font (size 1.27 1.27)) hide)
     )
@@
     )
     (property "Value" "Conn_01x02" (id 1) (at 269.24 99.06 0))
-    (property "Footprint" "" (id 2) (at 269.24 102.87 0)
+    (property "Footprint" "TerminalBlock_Euroclamp:MVE252-5-V" (id 2) (at 269.24 102.87 0)
       (effects (font (size 1.27 1.27)) hide)
     )
@@
     )
     (path "/31d80b0f-d224-41d0-81cd-261baf5b980a"
-      (reference "J6") (unit 1) (value "Conn_01x02") (footprint "")
+      (reference "J6") (unit 1) (value "Conn_01x02") (footprint "TerminalBlock_Euroclamp:MVE252-5-V")
     )
     (path "/b60df4de-2aac-440b-9e9f-b14c96d41684"
-      (reference "J7") (unit 1) (value "Conn_01x02") (footprint "")
+      (reference "J7") (unit 1) (value "Conn_01x02") (footprint "TerminalBlock_Euroclamp:MVE252-5-V")
     )
     (path "/00000000-0000-0000-0000-0000605d9623"
@@
     )
     (path "/09ebdf7c-8ad3-4ef7-b64a-85cf5a878a6e"
-      (reference "J9") (unit 1) (value "Conn_01x02") (footprint "")
+      (reference "J9") (unit 1) (value "Conn_01x02") (footprint "TerminalBlock_Euroclamp:MVE252-5-V")
     )
     (path "/2fc9e04d-6fab-47f1-b4f9-d0ede37b44c7"
-      (reference "J10") (unit 1) (value "Conn_01x02") (footprint "")
+      (reference "J10") (unit 1) (value "Conn_01x02") (footprint "TerminalBlock_Euroclamp:MVE252-5-V")
     )
     (path "/00000000-0000-0000-0000-0000601ff48e"
@@
     )
     (path "/540de89d-e0fc-4ad9-b0c3-47ecc3bb910c"
-      (reference "R23") (unit 1) (value "470R") (footprint "")
+      (reference "R23") (unit 1) (value "470R") (footprint "Resistor_SMD:R_0805_2012Metric")
     )
     (path "/0dd934c9-ce84-41aa-b51a-15c6f11b9b43"
-      (reference "R24") (unit 1) (value "470R") (footprint "")
+      (reference "R24") (unit 1) (value "470R") (footprint "Resistor_SMD:R_0805_2012Metric")
     )
     (path "/857c828a-990f-45e3-8d14-cc15748fc857"
