File: dc01.kicad_sch (KiCad schematic)
At the start: 83 parts, among them J1 USB_C_Receptacle_USB2.0, J10 Conn_01x02, J2 PROG/DEBUG, J3 Conn_01x06, J4 RJ12, J5 RJ12, J6 Conn_01x02, J7 Conn_01x02, J8 Conn_01x02, J9 Conn_01x02, K1 AZ850-5, K2 AZ850-5, Q1 2N7002, Q2 2N7002, SW1 SW_Push, SW2 SW_Push, SW3 MFP 113 D, U1 STM32F103C8Tx, U2 AMS1117-3.3, U3 PC817, U4 PC817, Y1 8 MHz

Commit message: Reorder schematics.
Connections:
- net GND: now also U1.8 (VSSA)
- no-connect marks 21 -> 20
Other:
- moved on the sheet: C8, C9, D1, D14, D2, D3, D4, H1, H2, H3, J10, J9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
