File: pcb/dc01.kicad_sch (KiCad schematic)
At the start: 83 parts, among them J1 USB_C_Receptacle_USB2.0, J10 Conn_01x02, J2 PROG/DEBUG, J3 Conn_01x06, J4 RJ12, J5 RJ12, J6 Conn_01x02, J7 Conn_01x02, J8 Conn_01x02, J9 Conn_01x02, K1 AZ850-5, K2 AZ850-5, Q1 2N7002, Q2 2N7002, SW1 SW_Push, SW2 SW_Push, SW3 MFP 113 D, U1 STM32F103C8Tx, U2 AMS1117-3.3, U3 PC817, U4 PC817, Y1 8 MHz

Commit message: Switch relay indication LEDs & resistors.
Connections:
- net GND: now also D12.1 (K), D13.1 (K); no longer R14.2, R15.2
- net REL1CTRL: now also R14.1; no longer D12.2 (A)
- net REL2CTRL: now also R15.1; no longer D13.2 (A)
- new net: D13.2 (A), R15.2
- new net: D12.2 (A), R14.2
Other:
- moved on the sheet: D12, D13, R14, R15
Changed lines of the file:
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@@
     (stroke (width 0) (type default) (color 0 0 0 0))
   )
-  (wire (pts (xy 266.7 147.32) (xy 266.7 149.86))
+  (wire (pts (xy 266.7 154.94) (xy 266.7 157.48))
     (stroke (width 0) (type default) (color 0 0 0 0))
   )
@@
     (stroke (width 0) (type default) (color 0 0 0 0))
   )
-  (wire (pts (xy 266.7 40.64) (xy 266.7 43.18))
+  (wire (pts (xy 266.7 48.26) (xy 266.7 50.8))
     (stroke (width 0) (type default) (color 0 0 0 0))
   )
@@
     (pin "2")
   )
-  (symbol (lib_id "Device:R") (at 266.7 153.67 0) (unit 1)
+  (symbol (lib_id "Device:R") (at 266.7 143.51 0) (unit 1)
     (in_bom yes) (on_board yes) (fields_autoplaced)
-    (property "Reference" "R15" (id 0) (at 268.478 152.8353 0)
+    (property "Reference" "R15" (id 0) (at 268.478 142.6753 0)
       (effects (font (size 1.27 1.27)) (justify left))
     )
-    (property "Value" "1k" (id 1) (at 268.478 155.3722 0)
+    (property "Value" "1k" (id 1) (at 268.478 145.2122 0)
       (effects (font (size 1.27 1.27)) (justify left))
     )
-    (property "Footprint" "Resistor_SMD:R_0805_2012Metric" (id 2) (at 264.922 153.67 90)
+    (property "Footprint" "Resistor_SMD:R_0805_2012Metric" (id 2) (at 264.922 143.51 90)
       (effects (font (size 1.27 1.27)) hide)
     )
-    (property "Datasheet" "~" (id 3) (at 266.7 153.67 0)
+    (property "Datasheet" "~" (id 3) (at 266.7 143.51 0)
       (effects (font (size 1.27 1.27)) hide)
     )
@@
     (pin "2")
   )
-  (symbol (lib_id "Device:R") (at 266.7 46.99 0) (unit 1)
+  (symbol (lib_id "Device:R") (at 266.7 36.83 0) (unit 1)
     (in_bom yes) (on_board yes) (fields_autoplaced)
-    (property "Reference" "R14" (id 0) (at 268.478 46.1553 0)
+    (property "Reference" "R14" (id 0) (at 268.478 35.9953 0)
       (effects (font (size 1.27 1.27)) (justify left))
     )
-    (property "Value" "1k" (id 1) (at 268.478 48.6922 0)
+    (property "Value" "1k" (id 1) (at 268.478 38.5322 0)
       (effects (font (size 1.27 1.27)) (justify left))
     )
-    (property "Footprint" "Resistor_SMD:R_0805_2012Metric" (id 2) (at 264.922 46.99 90)
+    (property "Footprint" "Resistor_SMD:R_0805_2012Metric" (id 2) (at 264.922 36.83 90)
       (effects (font (size 1.27 1.27)) hide)
     )
-    (property "Datasheet" "~" (id 3) (at 266.7 46.99 0)
+    (property "Datasheet" "~" (id 3) (at 266.7 36.83 0)
       (effects (font (size 1.27 1.27)) hide)
     )
@@
     (pin "2")
   )
-  (symbol (lib_id "Device:LED") (at 266.7 36.83 90) (unit 1)
+  (symbol (lib_id "Device:LED") (at 266.7 44.45 90) (unit 1)
     (in_bom yes) (on_board yes) (fields_autoplaced)
-    (property "Reference" "D12" (id 0) (at 269.621 37.5828 90)
+    (property "Reference" "D12" (id 0) (at 269.621 45.2028 90)
       (effects (font (size 1.27 1.27)) (justify right))
     )
-    (property "Value" "BLUE" (id 1) (at 269.621 40.1197 90)
+    (property "Value" "BLUE" (id 1) (at 269.621 47.7397 90)
       (effects (font (size 1.27 1.27)) (justify right))
     )
-    (property "Footprint" "LED_SMD:LED_0805_2012Metric" (id 2) (at 266.7 36.83 0)
+    (property "Footprint" "LED_SMD:LED_0805_2012Metric" (id 2) (at 266.7 44.45 0)
       (effects (font (size 1.27 1.27)) hide)
     )
-    (property "Datasheet" "~" (id 3) (at 266.7 36.83 0)
+    (property "Datasheet" "~" (id 3) (at 266.7 44.45 0)
       (effects (font (size 1.27 1.27)) hide)
     )
@@
     (pin "3")
   )
-  (symbol (lib_id "Device:LED") (at 266.7 143.51 90) (unit 1)
+  (symbol (lib_id "Device:LED") (at 266.7 151.13 90) (unit 1)
     (in_bom yes) (on_board yes) (fields_autoplaced)
-    (property "Reference" "D13" (id 0) (at 269.621 144.2628 90)
+    (property "Reference" "D13" (id 0) (at 269.621 151.8828 90)
       (effects (font (size 1.27 1.27)) (justify right))
     )
-    (property "Value" "BLUE" (id 1) (at 269.621 146.7997 90)
+    (property "Value" "BLUE" (id 1) (at 269.621 154.4197 90)
       (effects (font (size 1.27 1.27)) (justify right))
     )
-    (property "Footprint" "LED_SMD:LED_0805_2012Metric" (id 2) (at 266.7 143.51 0)
+    (property "Footprint" "LED_SMD:LED_0805_2012Metric" (id 2) (at 266.7 151.13 0)
       (effects (font (size 1.27 1.27)) hide)
     )
-    (property "Datasheet" "~" (id 3) (at 266.7 143.51 0)
+    (property "Datasheet" "~" (id 3) (at 266.7 151.13 0)
       (effects (font (size 1.27 1.27)) hide)
     )

Commit message: Divide into more sheets. Use relays in series.
Parts:
- removed C10, C11: 22u, Capacitor_SMD:C_0805_2012Metric, symbol Device:C
- removed D10, D6: GR, LED_SMD:LED_0805_2012Metric, symbol Device:LED
- removed D11, D5: 1N4148, Diode_THT:D_DO-35_SOD27_P7.62mm_Horizontal, symbol Diode:1N4148
- removed D12, D13: BLUE, LED_SMD:LED_0805_2012Metric, symbol Device:LED
- removed D8, D9: YEL, LED_SMD:LED_0805_2012Metric, symbol Device:LED
- removed F1, F2: 1A, Fuse:Fuse_1206_3216Metric, symbol Device:Polyfuse
- removed J4, J5: RJ12, Connector_RJ:RJ25_Wayconn_MJEA-660X1_Horizontal, symbol Connector:RJ12
- removed J6, J7: Conn_01x02, TerminalBlock_Euroclamp:MVE252-5-V, symbol Connector_Generic:Conn_01x02
- removed K1, K2: AZ850-5, Relay_THT:Relay_DPDT_FRT5, symbol Relay:AZ850-x
- removed Q1, Q2: 2N7002, Package_TO_SOT_SMD:SOT-23, symbol Transistor_FET:2N7002
- removed R10, R11, R12, R14, R15, R9: 1k, Resistor_SMD:R_0805_2012Metric, symbol Device:R
- removed R13, R8: 10k, Resistor_SMD:R_0805_2012Metric_Pad1.20x1.40mm_HandSolder, symbol Device:R
Connections:
- net REL1TESTIN2 is gone; now on net REL1CTRL: U1.20 (PB2)
- net REL1TESTOUT is gone; now on net REL2CTRL: U1.39 (PB3)
- net LED_GO: now also U1.22 (PB11); no longer U1.21 (PB10)
- net LED_STOP: now also U1.21 (PB10); no longer U1.22 (PB11)
- net REL1CTRL: no longer U1.18 (PB0)
- net REL2CTRL: no longer U1.40 (PB4)
- net BOOT0 renamed BOOT
- net REL1TESTIN1 renamed IO2DCC
- net REL2TESTIN1: no longer names the net of U1.41 (PB5)
- net REL2TESTIN2: no longer names the net of U1.42 (PB6)
- net REL2TESTOUT: no longer names the net of U1.43 (PB7)
- new net IO1DCC: U1.18 (PB0)
- new net RELCLOCK: U1.40 (PB4)
- no-connect marks 20 -> 21
Other:
- added sheet DCC cutting (cut.kicad_sch)
- added sheet Safe relay signal generation (safesig.kicad_sch)
- title: DCC cutter DC-01 -> DCC cutter DC-01 - overall schematics
- moved on the sheet: C1, C2, C3, C4, C5, C6, C7, C8, C9, D1, D14, D15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

Commit message: Fix ERC.
Connections:
- net OUT_ALERT: now also U1.41 (PB5); no longer U1.45 (PB8)
- net OUT_ON: now also U1.42 (PB6); no longer U1.46 (PB9)
- net SW_GO: now also U1.43 (PB7); no longer U1.14 (PA4)
- net SW_OVERRIDE: now also U1.46 (PB9); no longer U1.16 (PA6)
- net SW_STOP: now also U1.45 (PB8); no longer U1.15 (PA5)
- net RELCLOCK: no longer names the net of U1.40 (PB4)
- no-connect marks 21 -> 22
Other:
- sheet Safe relay signal generation ports: added none; removed CLKIN

Commit message: Add subschematics, add footprints.
Parts:
- D14: LCSC C84256 -> C2296
- R16, R18, R19: LCSC (none) -> C17414
- U3, U4: footprint Package_DIP:DIP-4_W7.62mm -> Package_DIP:DIP-4_W8.89mm_SMDSocket_LongPads
Changed lines of the file:
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@@
     (property "Reference" "U4" (id 0) (at 246.38 95.9952 0))
     (property "Value" "PC817" (id 1) (at 246.38 98.5321 0))
-    (property "Footprint" "Package_DIP:DIP-4_W7.62mm" (id 2) (at 241.3 108.585 0)
+    (property "Footprint" "Package_DIP:DIP-4_W8.89mm_SMDSocket_LongPads" (id 2) (at 241.3 108.585 0)
       (effects (font (size 1.27 1.27) italic) (justify left) hide)
     )
@@
       (effects (font (size 1.27 1.27)) hide)
     )
-    (property "LCSC" "C84256" (id 4) (at 76.2 165.735 0)
+    (property "LCSC" "C2296" (id 4) (at 76.2 165.735 0)
       (effects (font (size 1.27 1.27)) hide)
     )
@@
       (effects (font (size 1.27 1.27)) hide)
     )
+    (property "LCSC" "C17414" (id 4) (at 126.365 163.195 0)
+      (effects (font (size 1.27 1.27)) hide)
+    )
     (pin "1")
     (pin "2")
@@
     (property "Reference" "U3" (id 0) (at 246.38 82.0252 0))
     (property "Value" "PC817" (id 1) (at 246.38 84.5621 0))
-    (property "Footprint" "Package_DIP:DIP-4_W7.62mm" (id 2) (at 241.3 94.615 0)
+    (property "Footprint" "Package_DIP:DIP-4_W8.89mm_SMDSocket_LongPads" (id 2) (at 241.3 94.615 0)
       (effects (font (size 1.27 1.27) italic) (justify left) hide)
     )
@@
       (effects (font (size 1.27 1.27)) hide)
     )
+    (property "LCSC" "C17414" (id 4) (at 67.31 163.195 0)
+      (effects (font (size 1.27 1.27)) hide)
+    )
     (pin "1")
     (pin "2")
@@
     )
     (property "Datasheet" "~" (id 3) (at 102.235 163.195 0)
+      (effects (font (size 1.27 1.27)) hide)
+    )
+    (property "LCSC" "C17414" (id 4) (at 102.235 163.195 0)
       (effects (font (size 1.27 1.27)) hide)
     )
@@
     )
     (path "/7d37d309-375e-4a1a-8b3f-c3df19c8683d/aebce090-2588-4c08-a6e6-0462b5b5a4a2"
-      (reference "C10") (unit 1) (value "10n") (footprint "")
+      (reference "C10") (unit 1) (value "10n") (footprint "Capacitor_SMD:C_0805_2012Metric")
     )
     (path "/7d37d309-375e-4a1a-8b3f-c3df19c8683d/c1004a51-21ac-4aa8-ac25-e63aaf7c2964"
-      (reference "C11") (unit 1) (value "10n") (footprint "")
+      (reference "C11") (unit 1) (value "10n") (footprint "Capacitor_SMD:C_0805_2012Metric")
     )
     (path "/7d37d309-375e-4a1a-8b3f-c3df19c8683d/83e6089a-f759-41ad-baab-d58812cf65c4"
@@
     )
     (path "/2cf54f45-b5f3-43f0-9920-2b504cf8dc98/34f76e21-13df-4f85-b12f-e1c8eda553ec"
-      (reference "C14") (unit 1) (value "100n") (footprint "")
+      (reference "C14") (unit 1) (value "100n") (footprint "Capacitor_SMD:C_0805_2012Metric")
     )
     (path "/2cf54f45-b5f3-43f0-9920-2b504cf8dc98/8ce92fdc-7965-4ae1-a5fd-44c7419f2506"
-      (reference "C15") (unit 1) (value "100n") (footprint "")
+      (reference "C15") (unit 1) (value "100n") (footprint "Capacitor_SMD:C_0805_2012Metric")
     )
     (path "/2cf54f45-b5f3-43f0-9920-2b504cf8dc98/b8dffeb9-cc67-4d40-a361-76e8f03dbbc6"
-      (reference "C16") (unit 1) (value "100n") (footprint "")
+      (reference "C16") (unit 1) (value "100n") (footprint "Capacitor_SMD:C_0805_2012Metric")
     )
     (path "/00000000-0000-0000-0000-0000604f455e"
@@
     )
     (path "/7d37d309-375e-4a1a-8b3f-c3df19c8683d/a253db53-2d47-438f-9c9a-c957c233ec0b"
-      (reference "D5") (unit 1) (value "D_Bridge_+-AA") (footprint "")
+      (reference "D5") (unit 1) (value "D_Bridge_+-AA") (footprint "Rectifiers:S250")
     )
     (path "/7d37d309-375e-4a1a-8b3f-c3df19c8683d/43e0ddfe-9c81-46cc-9e22-6b2de1757565"
-      (reference "D6") (unit 1) (value "D_Bridge_+-AA") (footprint "")
+      (reference "D6") (unit 1) (value "D_Bridge_+-AA") (footprint "Rectifiers:S250")
     )
     (path "/00000000-0000-0000-0000-0000603f03f2"
@@
     )
     (path "/7d37d309-375e-4a1a-8b3f-c3df19c8683d/6ef5f09d-0848-43d3-a165-a95b7ecf252b"
-      (reference "R8") (unit 1) (value "10k") (footprint "")
+      (reference "R8") (unit 1) (value "10k") (footprint "Resistor_SMD:R_0805_2012Metric")
     )
     (path "/7d37d309-375e-4a1a-8b3f-c3df19c8683d/10f0245d-4826-40cb-846b-f5cb7cbfe5c0"
-      (reference "R9") (unit 1) (value "10k") (footprint "")
+      (reference "R9") (unit 1) (value "10k") (footprint "Resistor_SMD:R_0805_2012Metric")
     )
     (path "/7d37d309-375e-4a1a-8b3f-c3df19c8683d/7500c223-35d1-4477-a2e1-7e12e1f3ccca"
-      (reference "R10") (unit 1) (value "2k2") (footprint "")
+      (reference "R10") (unit 1) (value "2k2") (footprint "Resistor_SMD:R_0805_2012Metric")
     )
     (path "/7d37d309-375e-4a1a-8b3f-c3df19c8683d/cb45c5d3-3910-4096-9957-f6ec15489df2"
-      (reference "R11") (unit 1) (value "2k2") (footprint "")
+      (reference "R11") (unit 1) (value "2k2") (footprint "Resistor_SMD:R_0805_2012Metric")
     )
     (path "/7d37d309-375e-4a1a-8b3f-c3df19c8683d/221a9503-8351-4998-a6d6-f2f08edfe7ff"
-      (reference "R12") (unit 1) (value "1k") (footprint "")
+      (reference "R12") (unit 1) (value "1k") (footprint "Resistor_SMD:R_0805_2012Metric")
     )
     (path "/7d37d309-375e-4a1a-8b3f-c3df19c8683d/b731b4c6-38e5-42c0-9325-6b31d471d3a7"
-      (reference "R13") (unit 1) (value "1k") (footprint "")
+      (reference "R13") (unit 1) (value "1k") (footprint "Resistor_SMD:R_0805_2012Metric")
     )
     (path "/7d37d309-375e-4a1a-8b3f-c3df19c8683d/cc333350-f9d4-47f1-b805-772c14b2b012"
@@
     )
     (path "/7d37d309-375e-4a1a-8b3f-c3df19c8683d/1a059fb0-f439-4377-bce2-7ed866f60c96"
-      (reference "R15") (unit 1) (value "10k") (footprint "Resistor_SMD:R_0805_2012Metric_Pad1.20x1.40mm_HandSolder")
+      (reference "R15") (unit 1) (value "10k") (footprint "Resistor_SMD:R_0805_2012Metric")
     )
     (path "/d5411c03-6e71-4c73-a9f3-f764362d1dde"
@@
     )
     (path "/7d37d309-375e-4a1a-8b3f-c3df19c8683d/b8696f2e-79a4-4a43-9077-af50f79e44a3"
-      (reference "R25") (unit 1) (value "10k") (footprint "Resistor_SMD:R_0805_2012Metric_Pad1.20x1.40mm_HandSolder")
+      (reference "R25") (unit 1) (value "10k") (footprint "Resistor_SMD:R_0805_2012Metric")
     )
     (path "/7d37d309-375e-4a1a-8b3f-c3df19c8683d/41e71917-46a4-4506-8f54-4cf15d1abaee"
@@
     )
     (path "/2cf54f45-b5f3-43f0-9920-2b504cf8dc98/d81bf3c4-6f0c-42b3-9ca2-6d2ff89153d8"
-      (reference "R27") (unit 1) (value "47k") (footprint "")
+      (reference "R27") (unit 1) (value "47k") (footprint "Resistor_SMD:R_0805_2012Metric")
     )
     (path "/2cf54f45-b5f3-43f0-9920-2b504cf8dc98/dc2df260-7707-4aad-81ef-3b5d274d574b"
-      (reference "R28") (unit 1) (value "47k") (footprint "")
+      (reference "R28") (unit 1) (value "47k") (footprint "Resistor_SMD:R_0805_2012Metric")
     )
     (path "/857c828a-990f-45e3-8d14-cc15748fc857"
@@
     )
     (path "/8ddc6e36-5132-4854-afed-d9e2a402069f"
-      (reference "U3") (unit 1) (value "PC817") (footprint "Package_DIP:DIP-4_W7.62mm")
+      (reference "U3") (unit 1) (value "PC817") (footprint "Package_DIP:DIP-4_W8.89mm_SMDSocket_LongPads")
     )
     (path "/3f73a6bc-0684-4993-89dc-ae17a3d945e2"
-      (reference "U4") (unit 1) (value "PC817") (footprint "Package_DIP:DIP-4_W7.62mm")
+      (reference "U4") (unit 1) (value "PC817") (footprint "Package_DIP:DIP-4_W8.89mm_SMDSocket_LongPads")
     )
     (path "/7d37d309-375e-4a1a-8b3f-c3df19c8683d/0d300bf7-ea67-4841-9c62-0d5b70b4f5f5"
-      (reference "U5") (unit 1) (value "PC817") (footprint "Package_DIP:DIP-4_W7.62mm")
+      (reference "U5") (unit 1) (value "PC817") (footprint "Package_DIP:DIP-4_W8.89mm_SMDSocket_LongPads")
     )
     (path "/7d37d309-375e-4a1a-8b3f-c3df19c8683d/a30234d7-2082-4441-86e3-4347c37f0a5e"
-      (reference "U6") (unit 1) (value "PC817") (footprint "Package_DIP:DIP-4_W7.62mm")
+      (reference "U6") (unit 1) (value "PC817") (footprint "Package_DIP:DIP-4_W8.89mm_SMDSocket_LongPads")
     )
     (path "/2cf54f45-b5f3-43f0-9920-2b504cf8dc98/0eea7344-a7f2-4eca-bb02-37ab50dcd04c"
-      (reference "U7") (unit 1) (value "74HC123") (footprint "")
+      (reference "U7") (unit 1) (value "74HC123") (footprint "Package_SO:SOIC-16_3.9x9.9mm_P1.27mm")
     )
     (path "/2cf54f45-b5f3-43f0-9920-2b504cf8dc98/47c50aab-b180-4140-8490-703fcdeea0e3"
-      (reference "U7") (unit 2) (value "74HC123") (footprint "")
+      (reference "U7") (unit 2) (value "74HC123") (footprint "Package_SO:SOIC-16_3.9x9.9mm_P1.27mm")
     )
     (path "/2cf54f45-b5f3-43f0-9920-2b504cf8dc98/e419d987-00ce-40c7-b155-8c5dd9657cd3"
-      (reference "U7") (unit 3) (value "74HC123") (footprint "")
+      (reference "U7") (unit 3) (value "74HC123") (footprint "Package_SO:SOIC-16_3.9x9.9mm_P1.27mm")
     )
     (path "/00000000-0000-0000-0000-000060235da4"

Commit message: Use proper value for screw terminals.
Parts:
- J10, J9: value Conn_01x02 -> MVE252-5-V
Changed lines of the file:
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@@
       (effects (font (size 1.27 1.27)) (justify left))
     )
-    (property "Value" "Conn_01x02" (id 1) (at 266.192 89.9672 0)
+    (property "Value" "MVE252-5-V" (id 1) (at 266.192 89.9672 0)
       (effects (font (size 1.27 1.27)) (justify left))
     )
@@
       (effects (font (size 1.27 1.27)) (justify left))
     )
-    (property "Value" "Conn_01x02" (id 1) (at 266.192 103.9372 0)
+    (property "Value" "MVE252-5-V" (id 1) (at 266.192 103.9372 0)
       (effects (font (size 1.27 1.27)) (justify left))
     )
@@
     )
     (path "/7d37d309-375e-4a1a-8b3f-c3df19c8683d/2fcba7ba-df1c-4745-a2a2-d9d3b5c84860"
-      (reference "J6") (unit 1) (value "Conn_01x02") (footprint "TerminalBlock_Euroclamp:MVE252-5-V")
+      (reference "J6") (unit 1) (value "MVE252-5-V") (footprint "TerminalBlock_Euroclamp:MVE252-5-V")
     )
     (path "/7d37d309-375e-4a1a-8b3f-c3df19c8683d/4158d113-ab0f-4a93-aa7f-b745746d1045"
-      (reference "J7") (unit 1) (value "Conn_01x02") (footprint "TerminalBlock_Euroclamp:MVE252-5-V")
+      (reference "J7") (unit 1) (value "MVE252-5-V") (footprint "TerminalBlock_Euroclamp:MVE252-5-V")
     )
     (path "/00000000-0000-0000-0000-0000605d9623"
@@
     )
     (path "/09ebdf7c-8ad3-4ef7-b64a-85cf5a878a6e"
-      (reference "J9") (unit 1) (value "Conn_01x02") (footprint "TerminalBlock_Euroclamp:MVE252-5-V")
+      (reference "J9") (unit 1) (value "MVE252-5-V") (footprint "TerminalBlock_Euroclamp:MVE252-5-V")
     )
     (path "/2fc9e04d-6fab-47f1-b4f9-d0ede37b44c7"
-      (reference "J10") (unit 1) (value "Conn_01x02") (footprint "TerminalBlock_Euroclamp:MVE252-5-V")
+      (reference "J10") (unit 1) (value "MVE252-5-V") (footprint "TerminalBlock_Euroclamp:MVE252-5-V")
     )
     (path "/00000000-0000-0000-0000-0000601ff48e"

Commit message: Use MV132 as screw terminals.
Parts:
- J10, J9: value MVE252-5-V -> MV132; footprint TerminalBlock_Euroclamp:MVE252-5-V -> TerminalBlock_4Ucon:TerminalBlock_4Ucon_1x02_P3.50mm_Horizontal
Changed lines of the file:
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@@
       (effects (font (size 1.27 1.27)) (justify left))
     )
-    (property "Value" "MVE252-5-V" (id 1) (at 266.192 89.9672 0)
-      (effects (font (size 1.27 1.27)) (justify left))
-    )
-    (property "Footprint" "TerminalBlock_Euroclamp:MVE252-5-V" (id 2) (at 264.16 86.995 0)
+    (property "Value" "MV132" (id 1) (at 266.192 89.9672 0)
+      (effects (font (size 1.27 1.27)) (justify left))
+    )
+    (property "Footprint" "TerminalBlock_4Ucon:TerminalBlock_4Ucon_1x02_P3.50mm_Horizontal" (id 2) (at 264.16 86.995 0)
       (effects (font (size 1.27 1.27)) hide)
     )
@@
       (effects (font (size 1.27 1.27)) (justify left))
     )
-    (property "Value" "MVE252-5-V" (id 1) (at 266.192 103.9372 0)
-      (effects (font (size 1.27 1.27)) (justify left))
-    )
-    (property "Footprint" "TerminalBlock_Euroclamp:MVE252-5-V" (id 2) (at 264.16 100.965 0)
+    (property "Value" "MV132" (id 1) (at 266.192 103.9372 0)
+      (effects (font (size 1.27 1.27)) (justify left))
+    )
+    (property "Footprint" "TerminalBlock_4Ucon:TerminalBlock_4Ucon_1x02_P3.50mm_Horizontal" (id 2) (at 264.16 100.965 0)
       (effects (font (size 1.27 1.27)) hide)
     )
@@
     )
     (path "/7d37d309-375e-4a1a-8b3f-c3df19c8683d/2fcba7ba-df1c-4745-a2a2-d9d3b5c84860"
-      (reference "J6") (unit 1) (value "MVE252-5-V") (footprint "TerminalBlock_Euroclamp:MVE252-5-V")
+      (reference "J6") (unit 1) (value "MV132") (footprint "TerminalBlock_4Ucon:TerminalBlock_4Ucon_1x02_P3.50mm_Horizontal")
     )
     (path "/7d37d309-375e-4a1a-8b3f-c3df19c8683d/4158d113-ab0f-4a93-aa7f-b745746d1045"
-      (reference "J7") (unit 1) (value "MVE252-5-V") (footprint "TerminalBlock_Euroclamp:MVE252-5-V")
+      (reference "J7") (unit 1) (value "MV132") (footprint "TerminalBlock_4Ucon:TerminalBlock_4Ucon_1x02_P3.50mm_Horizontal")
     )
     (path "/00000000-0000-0000-0000-0000605d9623"
@@
     )
     (path "/09ebdf7c-8ad3-4ef7-b64a-85cf5a878a6e"
-      (reference "J9") (unit 1) (value "MVE252-5-V") (footprint "TerminalBlock_Euroclamp:MVE252-5-V")
+      (reference "J9") (unit 1) (value "MV132") (footprint "TerminalBlock_4Ucon:TerminalBlock_4Ucon_1x02_P3.50mm_Horizontal")
     )
     (path "/2fc9e04d-6fab-47f1-b4f9-d0ede37b44c7"
-      (reference "J10") (unit 1) (value "MVE252-5-V") (footprint "TerminalBlock_Euroclamp:MVE252-5-V")
+      (reference "J10") (unit 1) (value "MV132") (footprint "TerminalBlock_4Ucon:TerminalBlock_4Ucon_1x02_P3.50mm_Horizontal")
     )
     (path "/00000000-0000-0000-0000-0000601ff48e"
