File: pcb/dc01.kicad_sch (KiCad schematic)
At the start: 55 parts, among them J1 USB_C_Receptacle_USB2.0, J10 MV132, J2 PROG/DEBUG, J3 Conn_01x06, J8 Conn_01x02, J9 MV132, SW1 SW_Push, SW2 SW_Push, SW3 MFP 113 D, U1 STM32F103C8Tx, U2 AMS1117-3.3, U3 PC817, U4 PC817, Y1 8 MHz

Commit message: Draw & route part of PCB.
Connections:
- net USBD+: now also D7.6 (IO5); no longer D7.4 (IO3)
- net USBD-: now also D7.4 (IO3); no longer D7.6 (IO5)
Changed lines of the file:
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@@
   (junction (at 70.485 29.21) (diameter 0) (color 0 0 0 0)
   )
-  (junction (at 232.41 42.545) (diameter 0) (color 0 0 0 0)
-  )
   (junction (at 40.64 27.305) (diameter 0) (color 0 0 0 0)
   )
   (junction (at 76.2 186.055) (diameter 0) (color 0 0 0 0)
   )
+  (junction (at 237.49 42.545) (diameter 0) (color 0 0 0 0)
+  )
   (junction (at 94.615 52.07) (diameter 0) (color 0 0 0 0)
   )
+  (junction (at 232.41 45.085) (diameter 0) (color 0 0 0 0)
+  )
   (junction (at 52.705 186.055) (diameter 0) (color 0 0 0 0)
   )
@@
   )
   (junction (at 224.79 27.305) (diameter 0) (color 0 0 0 0)
-  )
-  (junction (at 237.49 45.085) (diameter 0) (color 0 0 0 0)
   )
   (junction (at 40.64 19.685) (diameter 0) (color 0 0 0 0)
@@
     (stroke (width 0) (type default) (color 0 0 0 0))
   )
+  (wire (pts (xy 226.06 42.545) (xy 237.49 42.545))
+    (stroke (width 0) (type default) (color 0 0 0 0))
+  )
   (wire (pts (xy 94.615 20.955) (xy 93.345 20.955))
     (stroke (width 0) (type default) (color 0 0 0 0))
@@
     (stroke (width 0) (type default) (color 0 0 0 0))
   )
-  (wire (pts (xy 232.41 47.625) (xy 232.41 42.545))
-    (stroke (width 0) (type default) (color 0 0 0 0))
-  )
   (wire (pts (xy 259.08 147.32) (xy 262.89 147.32))
     (stroke (width 0) (type default) (color 0 0 0 0))
@@
     (stroke (width 0) (type default) (color 0 0 0 0))
   )
-  (wire (pts (xy 247.65 45.085) (xy 237.49 45.085))
+  (wire (pts (xy 226.06 45.085) (xy 232.41 45.085))
     (stroke (width 0) (type default) (color 0 0 0 0))
   )
@@
     (stroke (width 0) (type default) (color 0 0 0 0))
   )
+  (wire (pts (xy 237.49 42.545) (xy 237.49 47.625))
+    (stroke (width 0) (type default) (color 0 0 0 0))
+  )
   (bus (pts (xy 107.315 132.715) (xy 107.315 136.525))
     (stroke (width 0) (type default) (color 0 0 0 0))
@@
     (stroke (width 0) (type default) (color 0 0 0 0))
   )
-  (wire (pts (xy 237.49 47.625) (xy 237.49 45.085))
-    (stroke (width 0) (type default) (color 0 0 0 0))
-  )
   (wire (pts (xy 236.22 106.045) (xy 236.22 92.075))
     (stroke (width 0) (type default) (color 0 0 0 0))
@@
     (stroke (width 0) (type default) (color 0 0 0 0))
   )
-  (wire (pts (xy 232.41 42.545) (xy 226.06 42.545))
-    (stroke (width 0) (type default) (color 0 0 0 0))
-  )
   (wire (pts (xy 85.725 92.71) (xy 104.775 92.71))
     (stroke (width 0) (type default) (color 0 0 0 0))
@@
     (stroke (width 0) (type default) (color 0 0 0 0))
   )
-  (wire (pts (xy 247.65 42.545) (xy 232.41 42.545))
+  (wire (pts (xy 247.65 42.545) (xy 237.49 42.545))
+    (stroke (width 0) (type default) (color 0 0 0 0))
+  )
+  (wire (pts (xy 232.41 45.085) (xy 232.41 47.625))
     (stroke (width 0) (type default) (color 0 0 0 0))
   )
@@
     (stroke (width 0) (type default) (color 0 0 0 0))
   )
-  (wire (pts (xy 237.49 45.085) (xy 226.06 45.085))
-    (stroke (width 0) (type default) (color 0 0 0 0))
-  )
   (wire (pts (xy 262.89 66.675) (xy 262.89 67.945))
     (stroke (width 0) (type default) (color 0 0 0 0))
@@
   )
   (wire (pts (xy 115.57 75.565) (xy 111.76 75.565))
+    (stroke (width 0) (type default) (color 0 0 0 0))
+  )
+  (wire (pts (xy 232.41 45.085) (xy 247.65 45.085))
     (stroke (width 0) (type default) (color 0 0 0 0))
   )
@@
     )
     (path "/7d37d309-375e-4a1a-8b3f-c3df19c8683d/1a831434-d82a-437c-a810-d2429e3e53d0"
-      (reference "D10") (unit 1) (value "1N4148") (footprint "Diode_THT:D_DO-35_SOD27_P7.62mm_Horizontal")
+      (reference "D10") (unit 1) (value "1N4148") (footprint "Diode_SMD:D_0805_2012Metric_Pad1.15x1.40mm_HandSolder")
     )
     (path "/7d37d309-375e-4a1a-8b3f-c3df19c8683d/065d9eae-2017-428e-9561-ae4591beda84"
-      (reference "D11") (unit 1) (value "1N4148") (footprint "Diode_THT:D_DO-35_SOD27_P7.62mm_Horizontal")
+      (reference "D11") (unit 1) (value "1N4148") (footprint "Diode_SMD:D_0805_2012Metric_Pad1.15x1.40mm_HandSolder")
     )
     (path "/7d37d309-375e-4a1a-8b3f-c3df19c8683d/634a928d-3c0e-46a8-8685-72733a9d516c"

Commit message: Minor silkscreen tweaks.
Parts:
- H1, H2, H3: symbol Mechanical:MountingHole_Pad -> Mechanical:MountingHole
- renumbered TP6 to TP1
Connections:
- no-connect marks 22 -> 19
Other:
- moved on the sheet: TP1
Changed lines of the file:
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@@
   (no_connect (at 85.725 59.69))
   (no_connect (at 52.705 67.31))
-  (no_connect (at 151.765 177.8))
-  (no_connect (at 154.305 185.42))
   (no_connect (at 85.725 54.61))
   (no_connect (at 242.57 47.625))
@@
   (no_connect (at 246.38 144.78))
   (no_connect (at 270.51 65.405))
-  (no_connect (at 156.845 177.8))
   (no_connect (at 247.65 55.245))
   (no_connect (at 68.58 174.625))
@@
     (stroke (width 0) (type default) (color 0 0 0 0))
   )
-  (text "JLCPCB tooling holes" (at 164.465 189.23 180)
+  (text "JLCPCB tooling holes" (at 163.195 174.625 180)
     (effects (font (size 1.27 1.27)) (justify right bottom))
   )
@@
     (pin "2")
   )
-  (symbol (lib_id "Connector:TestPoint") (at 154.305 160.02 0) (mirror y) (unit 1)
-    (in_bom yes) (on_board yes)
-    (property "Reference" "TP6" (id 0) (at 152.8318 157.0228 0)
-      (effects (font (size 1.27 1.27)) (justify left))
-    )
-    (property "Value" "TestPoint" (id 1) (at 152.8318 159.3342 0)
-      (effects (font (size 1.27 1.27)) (justify left))
-    )
-    (property "Footprint" "TestPoint:TestPoint_Loop_D3.50mm_Drill1.4mm_Beaded" (id 2) (at 149.225 160.02 0)
-      (effects (font (size 1.27 1.27)) hide)
-    )
-    (property "Datasheet" "~" (id 3) (at 149.225 160.02 0)
-      (effects (font (size 1.27 1.27)) hide)
-    )
-    (property "JLCPCB_IGNORE" "true" (id 4) (at 154.305 160.02 0)
-      (effects (font (size 1.27 1.27)) hide)
-    )
-    (pin "1")
-  )
-  (symbol (lib_id "power:GND") (at 154.305 160.02 0) (mirror y) (unit 1)
-    (in_bom yes) (on_board yes)
-    (property "Reference" "#PWR0104" (id 0) (at 154.305 166.37 0)
-      (effects (font (size 1.27 1.27)) hide)
-    )
-    (property "Value" "GND" (id 1) (at 154.178 164.4142 0))
-    (property "Footprint" "" (id 2) (at 154.305 160.02 0)
-      (effects (font (size 1.27 1.27)) hide)
-    )
-    (property "Datasheet" "" (id 3) (at 154.305 160.02 0)
+  (symbol (lib_id "Connector:TestPoint") (at 153.035 145.415 0) (mirror y) (unit 1)
+    (in_bom yes) (on_board yes)
+    (property "Reference" "TP1" (id 0) (at 151.5618 142.4178 0)
+      (effects (font (size 1.27 1.27)) (justify left))
+    )
+    (property "Value" "TestPoint" (id 1) (at 151.5618 144.7292 0)
+      (effects (font (size 1.27 1.27)) (justify left))
+    )
+    (property "Footprint" "TestPoint:TestPoint_Loop_D3.50mm_Drill1.4mm_Beaded" (id 2) (at 147.955 145.415 0)
+      (effects (font (size 1.27 1.27)) hide)
+    )
+    (property "Datasheet" "~" (id 3) (at 147.955 145.415 0)
+      (effects (font (size 1.27 1.27)) hide)
+    )
+    (property "JLCPCB_IGNORE" "true" (id 4) (at 153.035 145.415 0)
+      (effects (font (size 1.27 1.27)) hide)
+    )
+    (pin "1")
+  )
+  (symbol (lib_id "power:GND") (at 153.035 145.415 0) (mirror y) (unit 1)
+    (in_bom yes) (on_board yes)
+    (property "Reference" "#PWR0104" (id 0) (at 153.035 151.765 0)
+      (effects (font (size 1.27 1.27)) hide)
+    )
+    (property "Value" "GND" (id 1) (at 152.908 149.8092 0))
+    (property "Footprint" "" (id 2) (at 153.035 145.415 0)
+      (effects (font (size 1.27 1.27)) hide)
+    )
+    (property "Datasheet" "" (id 3) (at 153.035 145.415 0)
       (effects (font (size 1.27 1.27)) hide)
     )
@@
     (pin "2")
   )
-  (symbol (lib_id "Mechanical:MountingHole_Pad") (at 151.765 175.26 0) (mirror y) (unit 1)
-    (in_bom yes) (on_board yes)
-    (property "Reference" "H2" (id 0) (at 149.225 171.4754 0)
-      (effects (font (size 1.27 1.27)) (justify left))
-    )
-    (property "Value" "-" (id 1) (at 149.225 173.7868 0)
-      (effects (font (size 1.27 1.27)) (justify left))
-    )
-    (property "Footprint" "jlcpcb_tooling_holes:jlcpcb_tooling_holes" (id 2) (at 151.765 175.26 0)
-      (effects (font (size 1.27 1.27)) hide)
-    )
-    (property "Datasheet" "~" (id 3) (at 151.765 175.26 0)
-      (effects (font (size 1.27 1.27)) hide)
-    )
-    (property "JLCPCB_IGNORE" "true" (id 4) (at 151.765 175.26 0)
-      (effects (font (size 1.27 1.27)) hide)
-    )
-    (pin "1")
-  )
-  (symbol (lib_id "Mechanical:MountingHole_Pad") (at 156.845 175.26 0) (unit 1)
-    (in_bom yes) (on_board yes)
-    (property "Reference" "H1" (id 0) (at 159.385 171.45 0)
-      (effects (font (size 1.27 1.27)) (justify left))
-    )
-    (property "Value" "-" (id 1) (at 159.385 173.99 0)
-      (effects (font (size 1.27 1.27)) (justify left))
-    )
-    (property "Footprint" "jlcpcb_tooling_holes:jlcpcb_tooling_holes" (id 2) (at 156.845 175.26 0)
-      (effects (font (size 1.27 1.27)) hide)
-    )
-    (property "Datasheet" "~" (id 3) (at 156.845 175.26 0)
-      (effects (font (size 1.27 1.27)) hide)
-    )
-    (property "JLCPCB_IGNORE" "true" (id 4) (at 156.845 175.26 0)
-      (effects (font (size 1.27 1.27)) hide)
-    )
-    (pin "1")
-  )
-  (symbol (lib_id "Mechanical:MountingHole_Pad") (at 154.305 182.88 0) (mirror y) (unit 1)
-    (in_bom yes) (on_board yes)
-    (property "Reference" "H3" (id 0) (at 151.765 181.6354 0)
-      (effects (font (size 1.27 1.27)) (justify left))
-    )
-    (property "Value" "-" (id 1) (at 151.765 183.9468 0)
-      (effects (font (size 1.27 1.27)) (justify left))
-    )
-    (property "Footprint" "jlcpcb_tooling_holes:jlcpcb_tooling_holes" (id 2) (at 154.305 182.88 0)
-      (effects (font (size 1.27 1.27)) hide)
-    )
-    (property "Datasheet" "~" (id 3) (at 154.305 182.88 0)
-      (effects (font (size 1.27 1.27)) hide)
-    )
-    (property "JLCPCB_IGNORE" "true" (id 4) (at 154.305 182.88 0)
-      (effects (font (size 1.27 1.27)) hide)
-    )
-    (pin "1")
+  (symbol (lib_id "Mechanical:MountingHole") (at 149.86 161.29 0) (mirror y) (unit 1)
+    (in_bom yes) (on_board yes)
+    (property "Reference" "H2" (id 0) (at 147.32 157.5054 0)
+      (effects (font (size 1.27 1.27)) (justify left))
+    )
+    (property "Value" "-" (id 1) (at 147.32 159.8168 0)
+      (effects (font (size 1.27 1.27)) (justify left))
+    )
+    (property "Footprint" "jlcpcb_tooling_holes:jlcpcb_tooling_holes" (id 2) (at 149.86 161.29 0)
+      (effects (font (size 1.27 1.27)) hide)
+    )
+    (property "Datasheet" "~" (id 3) (at 149.86 161.29 0)
+      (effects (font (size 1.27 1.27)) hide)
+    )
+    (property "JLCPCB_IGNORE" "true" (id 4) (at 149.86 161.29 0)
+      (effects (font (size 1.27 1.27)) hide)
+    )
+  )
+  (symbol (lib_id "Mechanical:MountingHole") (at 156.21 161.29 0) (unit 1)
+    (in_bom yes) (on_board yes)
+    (property "Reference" "H1" (id 0) (at 158.75 157.48 0)
+      (effects (font (size 1.27 1.27)) (justify left))
+    )
+    (property "Value" "-" (id 1) (at 158.75 160.02 0)
+      (effects (font (size 1.27 1.27)) (justify left))
+    )
+    (property "Footprint" "jlcpcb_tooling_holes:jlcpcb_tooling_holes" (id 2) (at 156.21 161.29 0)
+      (effects (font (size 1.27 1.27)) hide)
+    )
+    (property "Datasheet" "~" (id 3) (at 156.21 161.29 0)
+      (effects (font (size 1.27 1.27)) hide)
+    )
+    (property "JLCPCB_IGNORE" "true" (id 4) (at 156.21 161.29 0)
+      (effects (font (size 1.27 1.27)) hide)
+    )
+  )
+  (symbol (lib_id "Mechanical:MountingHole") (at 153.035 168.275 0) (mirror y) (unit 1)
+    (in_bom yes) (on_board yes)
+    (property "Reference" "H3" (id 0) (at 150.495 167.0304 0)
+      (effects (font (size 1.27 1.27)) (justify left))
+    )
+    (property "Value" "-" (id 1) (at 150.495 169.3418 0)
+      (effects (font (size 1.27 1.27)) (justify left))
+    )
+    (property "Footprint" "jlcpcb_tooling_holes:jlcpcb_tooling_holes" (id 2) (at 153.035 168.275 0)
+      (effects (font (size 1.27 1.27)) hide)
+    )
+    (property "Datasheet" "~" (id 3) (at 153.035 168.275 0)
+      (effects (font (size 1.27 1.27)) hide)
+    )
+    (property "JLCPCB_IGNORE" "true" (id 4) (at 153.035 168.275 0)
+      (effects (font (size 1.27 1.27)) hide)
+    )
   )
   (symbol (lib_id "Connector_Generic:Conn_01x02") (at 264.16 86.995 0) (unit 1)
@@
     (pin "2")
   )
+  (symbol (lib_id "Graphic:Logo_Open_Hardware_Small") (at 168.275 190.5 0) (unit 1)
+    (in_bom yes) (on_board yes) (fields_autoplaced)
+    (property "Reference" "#LOGO1" (id 0) (at 168.275 183.515 0)
+      (effects (font (size 1.27 1.27)) hide)
+    )
+    (property "Value" "Logo_Open_Hardware_Small" (id 1) (at 168.275 196.215 0)
+      (effects (font (size 1.27 1.27)) hide)
+    )
+    (property "Footprint" "" (id 2) (at 168.275 190.5 0)
+      (effects (font (size 1.27 1.27)) hide)
+    )
+    (property "Datasheet" "~" (id 3) (at 168.275 190.5 0)
+      (effects (font (size 1.27 1.27)) hide)
+    )
+  )
   (symbol (lib_id "power:+3V3") (at 126.365 159.385 0) (unit 1)
     (in_bom yes) (on_board yes)
@@
       (reference "#FLG02") (unit 1) (value "PWR_FLAG") (footprint "")
     )
+    (path "/b3cb03fd-b6c9-4cba-a099-f1921a28b789"
+      (reference "#LOGO1") (unit 1) (value "Logo_Open_Hardware_Small") (footprint "")
+    )
     (path "/00000000-0000-0000-0000-000060338237"
       (reference "#PWR01") (unit 1) (value "GND") (footprint "")
@@
     )
     (path "/00000000-0000-0000-0000-0000604f6742"
-      (reference "TP6") (unit 1) (value "TestPoint") (footprint "TestPoint:TestPoint_Loop_D3.50mm_Drill1.4mm_Beaded")
+      (reference "TP1") (unit 1) (value "TestPoint") (footprint "TestPoint:TestPoint_Loop_D3.50mm_Drill1.4mm_Beaded")
     )
     (path "/00000000-0000-0000-0000-0000601d7b7c"

Commit message: Add LCSCs.
Parts:
- J10, J9, SW1, SW2, SW3: JLCPCB_IGNORE (none) -> true
- R23, R24: LCSC (none) -> C17710
- U3, U4: LCSC (none) -> C106900
Changed lines of the file:
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@@
+      (effects (font (size 1.27 1.27)) hide)
+    )
+    (property "JLCPCB_IGNORE" "true" (id 4) (at 264.16 86.995 0)
       (effects (font (size 1.27 1.27)) hide)
     )
@@
       (effects (font (size 1.27 1.27)) hide)
     )
+    (property "LCSC" "C17710" (id 4) (at 229.87 100.965 0)
+      (effects (font (size 1.27 1.27)) hide)
+    )
     (pin "1")
     (pin "2")
@@
     )
     (property "Datasheet" "~" (id 3) (at 117.475 175.895 0)
+      (effects (font (size 1.27 1.27)) hide)
+    )
+    (property "JLCPCB_IGNORE" "true" (id 4) (at 122.555 175.895 0)
       (effects (font (size 1.27 1.27)) hide)
     )
@@
     )
     (property "Datasheet" "~" (id 3) (at 264.16 100.965 0)
+      (effects (font (size 1.27 1.27)) hide)
+    )
+    (property "JLCPCB_IGNORE" "true" (id 4) (at 264.16 100.965 0)
       (effects (font (size 1.27 1.27)) hide)
     )
@@
       (effects (font (size 1.27 1.27)) (justify left) hide)
     )
+    (property "LCSC" "C106900" (id 4) (at 246.38 103.505 0)
+      (effects (font (size 1.27 1.27)) hide)
+    )
     (pin "1")
     (pin "2")
@@
       (effects (font (size 1.27 1.27)) hide)
     )
+    (property "LCSC" "C17710" (id 4) (at 229.87 86.995 0)
+      (effects (font (size 1.27 1.27)) hide)
+    )
     (pin "1")
     (pin "2")
@@
       (effects (font (size 1.27 1.27)) hide)
     )
+    (property "JLCPCB_IGNORE" "true" (id 4) (at 66.04 179.705 0)
+      (effects (font (size 1.27 1.27)) hide)
+    )
     (pin "1")
     (pin "2")
@@
     )
     (property "Datasheet" "~" (id 3) (at 93.345 175.895 0)
+      (effects (font (size 1.27 1.27)) hide)
+    )
+    (property "JLCPCB_IGNORE" "true" (id 4) (at 98.425 175.895 0)
       (effects (font (size 1.27 1.27)) hide)
     )
@@
       (effects (font (size 1.27 1.27)) (justify left) hide)
     )
-    (pin "1")
+    (property "LCSC" "C106900" (id 4) (at 246.38 89.535 0)
+      (effects (font (size 1.27 1.27)) hide)
+    )
+    (pin "1")

Commit message: Do not use 2 different types of diodes.
Parts:
- C8: LCSC C45783 -> C15850
Changed lines of the file:
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@@
       (effects (font (size 1.27 1.27)) hide)
     )
-    (property "LCSC" "C45783" (id 4) (at 189.865 43.18 0)
+    (property "LCSC" "C15850" (id 4) (at 189.865 43.18 0)
       (effects (font (size 1.27 1.27)) hide)
     )
@@
     )
     (path "/7d37d309-375e-4a1a-8b3f-c3df19c8683d/1a831434-d82a-437c-a810-d2429e3e53d0"
-      (reference "D10") (unit 1) (value "1N4148") (footprint "Diode_SMD:D_0805_2012Metric_Pad1.15x1.40mm_HandSolder")
+      (reference "D10") (unit 1) (value "1N5819") (footprint "Diode_SMD:D_SOD-123")
     )
     (path "/7d37d309-375e-4a1a-8b3f-c3df19c8683d/065d9eae-2017-428e-9561-ae4591beda84"
-      (reference "D11") (unit 1) (value "1N4148") (footprint "Diode_SMD:D_0805_2012Metric_Pad1.15x1.40mm_HandSolder")
+      (reference "D11") (unit 1) (value "1N5819") (footprint "Diode_SMD:D_SOD-123")
     )
     (path "/7d37d309-375e-4a1a-8b3f-c3df19c8683d/634a928d-3c0e-46a8-8685-72733a9d516c"

Commit message: Conn → screw terminals.
Parts:
- J10, J9: symbol Connector_Generic:Conn_01x02 -> Connector:Screw_Terminal_01x02
Changed lines of the file:
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@@
     )
   )
-  (symbol (lib_id "Connector_Generic:Conn_01x02") (at 264.16 86.995 0) (unit 1)
+  (symbol (lib_id "Connector:Screw_Terminal_01x02") (at 264.16 86.995 0) (unit 1)
     (in_bom yes) (on_board yes) (fields_autoplaced)
     (property "Reference" "J9" (id 0) (at 266.192 87.4303 0)
@@
     (pin "1")
   )
-  (symbol (lib_id "Connector_Generic:Conn_01x02") (at 264.16 100.965 0) (unit 1)
+  (symbol (lib_id "Connector:Screw_Terminal_01x02") (at 264.16 100.965 0) (unit 1)
     (in_bom yes) (on_board yes) (fields_autoplaced)
     (property "Reference" "J10" (id 0) (at 266.192 101.4003 0)

Commit message: Tweak resistor values for LEDs.
Parts:
- R21, R3: value 1k -> 10k; LCSC C17513 -> C17414
- R7: value 1k -> 2k2; LCSC C17513 -> C17520
Changed lines of the file:
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@@
       (effects (font (size 1.27 1.27)) (justify right))
     )
-    (property "Value" "1k" (id 1) (at 24.257 171.958 0)
+    (property "Value" "10k" (id 1) (at 24.257 171.958 0)
       (effects (font (size 1.27 1.27)) (justify right))
     )
@@
       (effects (font (size 1.27 1.27)) hide)
     )
-    (property "LCSC" "C17513" (id 4) (at 26.035 170.815 0)
+    (property "LCSC" "C17414" (id 4) (at 26.035 170.815 0)
       (effects (font (size 1.27 1.27)) hide)
     )
@@
       (effects (font (size 1.27 1.27)) (justify right))
     )
-    (property "Value" "1k" (id 1) (at 50.927 171.958 0)
+    (property "Value" "2k2" (id 1) (at 50.927 171.958 0)
       (effects (font (size 1.27 1.27)) (justify right))
     )
@@
       (effects (font (size 1.27 1.27)) hide)
     )
-    (property "LCSC" "C17513" (id 4) (at 52.705 170.815 0)
+    (property "LCSC" "C17520" (id 4) (at 52.705 170.815 0)
       (effects (font (size 1.27 1.27)) hide)
     )
@@
       (effects (font (size 1.27 1.27)) (justify right))
     )
-    (property "Value" "1k" (id 1) (at 90.297 171.958 0)
+    (property "Value" "10k" (id 1) (at 90.297 171.958 0)
       (effects (font (size 1.27 1.27)) (justify right))
     )
@@
       (effects (font (size 1.27 1.27)) hide)
     )
-    (property "LCSC" "C17513" (id 4) (at 92.075 170.815 0)
+    (property "LCSC" "C17414" (id 4) (at 92.075 170.815 0)
       (effects (font (size 1.27 1.27)) hide)
     )
@@
     )
     (path "/00000000-0000-0000-0000-00006086b397"
-      (reference "R3") (unit 1) (value "1k") (footprint "Resistor_SMD:R_0805_2012Metric")
+      (reference "R3") (unit 1) (value "10k") (footprint "Resistor_SMD:R_0805_2012Metric")
     )
     (path "/00000000-0000-0000-0000-000060229ef9"
@@
     )
     (path "/00000000-0000-0000-0000-00006086dbf4"
-      (reference "R7") (unit 1) (value "1k") (footprint "Resistor_SMD:R_0805_2012Metric")
+      (reference "R7") (unit 1) (value "2k2") (footprint "Resistor_SMD:R_0805_2012Metric")
     )
     (path "/7d37d309-375e-4a1a-8b3f-c3df19c8683d/6ef5f09d-0848-43d3-a165-a95b7ecf252b"
@@
     )
     (path "/7d37d309-375e-4a1a-8b3f-c3df19c8683d/cc333350-f9d4-47f1-b805-772c14b2b012"
-      (reference "R14") (unit 1) (value "1k") (footprint "Resistor_SMD:R_0805_2012Metric")
+      (reference "R14") (unit 1) (value "2k2") (footprint "Resistor_SMD:R_0805_2012Metric")
     )
     (path "/7d37d309-375e-4a1a-8b3f-c3df19c8683d/1a059fb0-f439-4377-bce2-7ed866f60c96"
@@
     )
     (path "/90e05316-6b44-4ac4-bc5c-e352392b2de3"
-      (reference "R21") (unit 1) (value "1k") (footprint "Resistor_SMD:R_0805_2012Metric")
+      (reference "R21") (unit 1) (value "10k") (footprint "Resistor_SMD:R_0805_2012Metric")
     )
     (path "/aa3da26d-068f-4c11-accd-793535927677"
@@
     )
     (path "/7d37d309-375e-4a1a-8b3f-c3df19c8683d/41e71917-46a4-4506-8f54-4cf15d1abaee"
-      (reference "R26") (unit 1) (value "1k") (footprint "Resistor_SMD:R_0805_2012Metric")
+      (reference "R26") (unit 1) (value "2k2") (footprint "Resistor_SMD:R_0805_2012Metric")
     )
     (path "/2cf54f45-b5f3-43f0-9920-2b504cf8dc98/d81bf3c4-6f0c-42b3-9ca2-6d2ff89153d8"
