File: pcb/dc01.kicad_sch (KiCad schematic)
At the start: 55 parts, among them J1 USB_C_Receptacle_USB2.0, J10 MV132, J2 PROG/DEBUG, J3 Conn_01x06, J8 Conn_01x02, J9 MV132, SW1 SW_Push, SW2 SW_Push, SW3 MFP 113 D, U1 STM32F103C8Tx, U2 AMS1117-3.3, U3 PC817, U4 PC817, Y1 8 MHz

Commit message: Switch active-alert outputs.
Connections:
- net OUT_ALERT: now also R24.1; no longer R23.1
- net OUT_ON: now also R23.1; no longer R24.1
Changed lines of the file:
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@@
     )
   )
-  (global_label "OUT_ALERT" (shape input) (at 223.52 86.995 180) (fields_autoplaced)
+  (global_label "OUT_ALERT" (shape input) (at 223.52 100.965 180) (fields_autoplaced)
     (effects (font (size 1.27 1.27)) (justify right))
-    (property "Intersheet References" "${INTERSHEET_REFS}" (id 0) (at 211.0963 86.9156 0)
+    (property "Intersheet References" "${INTERSHEET_REFS}" (id 0) (at 211.0963 100.8856 0)
       (effects (font (size 1.27 1.27)) (justify right) hide)
     )
@@
     )
   )
-  (global_label "OUT_ON" (shape input) (at 223.52 100.965 180) (fields_autoplaced)
+  (global_label "OUT_ON" (shape input) (at 223.52 86.995 180) (fields_autoplaced)
     (effects (font (size 1.27 1.27)) (justify right))
-    (property "Intersheet References" "${INTERSHEET_REFS}" (id 0) (at 213.9387 100.8856 0)
+    (property "Intersheet References" "${INTERSHEET_REFS}" (id 0) (at 213.9387 86.9156 0)
       (effects (font (size 1.27 1.27)) (justify right) hide)
     )
