File: pcb/dc01.kicad_pcb (KiCad board)
At the start: 2 copper layers, 76 x 84 mm, 76 parts, among them J1 USB_C_Receptacle_USB2.0, J2 PROG/DEBUG, J3 Conn_01x06, J4 RJ12, J5 RJ12, J6 Screw_Terminal_01x02, J7 Screw_Terminal_01x02, J8 Conn_01x02, U1 STM32F103C8Tx, U2 AMS1117-3.3, U3 ADM2483xRW, U4 ADUM1250, U6 LM78M05_TO252, U7 INA219AxDCN, Y1 8 MHz

Commit message: Clean up PCB (from MTB-USB v4).
Parts:
- removed C17: 470p, Capacitor_THT:C_Disc_D12.5mm_W5.0mm_P10.00mm
- removed JP5, JP6: SJ_2_Open, Jumper:SolderJumper-2_P1.3mm_Open_RoundedPad1.0x1.5mm
- removed JP7: SJ3_Bridged12, Jumper:SolderJumper-3_P1.3mm_Bridged12_RoundedPad1.0x1.5mm_NumberLabels
- removed PS1: AM2D-0505SZ, Converter_DCDC:Converter_DCDC_XP_POWER-IHxxxxS_THT
- removed TP1, TP2, TP3, TP4, TP5: TestPoint, TestPoint:TestPoint_Pad_D1.0mm
- removed TP7: TestPoint, TestPoint:TestPoint_Loop_D3.50mm_Drill1.4mm_Beaded
- added D10: 1N4148, Diode_THT:D_DO-35_SOD27_P7.62mm_Horizontal, F.Cu at (63.0, 72.4)
- added D11: 1N4148, Diode_THT:D_DO-35_SOD27_P7.62mm_Horizontal, F.Cu at (63.0, 68.8)
- added D12: BLUE, LED_SMD:LED_0805_2012Metric, F.Cu at (59.6, 88.6)
- added D13: BLUE, LED_SMD:LED_0805_2012Metric, F.Cu at (59.6, 85.6)
- added D14: YEL, LED_SMD:LED_0805_2012Metric, F.Cu at (40.3, 112.6)
- added D15: GR, LED_SMD:LED_0805_2012Metric, F.Cu at (40.3, 115.6)
- added D16: RED, LED_SMD:LED_0805_2012Metric, F.Cu at (44.7, 115.2)
- added D17: 1N5819, Diode_SMD:D_SOD-123, F.Cu at (70.1, 75.8)
- added D18: 1N5819, Diode_SMD:D_SOD-123, F.Cu at (54.5, 85.0)
- added D19: 1N5819, Diode_SMD:D_SOD-123, F.Cu at (75.1, 68.7)
- added D20: 1N5819, Diode_SMD:D_SOD-123, F.Cu at (75.1, 72.1)
- added D21: 1N5819, Diode_SMD:D_SOD-123, F.Cu at (64.3, 75.8)
- added D22: 1N5819, Diode_SMD:D_SOD-123, F.Cu at (54.5, 88.4)
- added D9: GR, LED_SMD:LED_0805_2012Metric, F.Cu at (53.9, 91.5)
- added F1: 1A, Fuse:Fuse_1206_3216Metric, F.Cu at (64.2, 82.4)
- added F2: 1A, Fuse:Fuse_1206_3216Metric, F.Cu at (64.2, 79.1)
- added J10: MV132, TerminalBlock_4Ucon:TerminalBlock_4Ucon_1x02_P3.50mm_Horizontal, F.Cu at (63.7, 100.5)
- added J9: MV132, TerminalBlock_4Ucon:TerminalBlock_4Ucon_1x02_P3.50mm_Horizontal, F.Cu at (51.7, 109.1)
- added K1: AZ850-5, Relay_THT:Relay_DPDT_FRT5, F.Cu at (40.1, 70.1)
- added K2: AZ850-5, Relay_THT:Relay_DPDT_FRT5, F.Cu at (51.8, 70.1)
- added Q1: 2N7002, Package_TO_SOT_SMD:SOT-23, F.Cu at (80.4, 69.3)
- added Q2: 2N7002, Package_TO_SOT_SMD:SOT-23, F.Cu at (69.5, 79.7)
- added R19: 10k, Resistor_SMD:R_0805_2012Metric, F.Cu at (65.0, 106.6)
- added R20: 1k, Resistor_SMD:R_0805_2012Metric, F.Cu at (60.5, 106.6)
- added R21: 1k, Resistor_SMD:R_0805_2012Metric, F.Cu at (72.5, 97.6)
- added R22: 1k, Resistor_SMD:R_0805_2012Metric, F.Cu at (60.5, 109.6)
- added R23: 470R, Resistor_SMD:R_0805_2012Metric, F.Cu at (53.6, 115.2)
- added R24: 470R, Resistor_SMD:R_0805_2012Metric, F.Cu at (49.1, 115.2)
- added R25: 10k, Resistor_SMD:R_0805_2012Metric, F.Cu at (44.7, 91.6)
- added R26: 1k, Resistor_SMD:R_0805_2012Metric, F.Cu at (64.0, 85.5)
- added R27: 47k, Resistor_SMD:R_0805_2012Metric, F.Cu at (89.6, 68.5)
- added R28: 47k, Resistor_SMD:R_0805_2012Metric, F.Cu at (89.6, 71.5)
- added R29: 1k, Resistor_SMD:R_0805_2012Metric, F.Cu at (49.1, 91.6)
- added R30: 1k, Resistor_SMD:R_0805_2012Metric, F.Cu at (40.2, 91.6)
- added SW1: SW_Push, Button_Switch_THT:SW_PUSH_6mm_H4.3mm, F.Cu at (52.0, 98.1)
- added SW2: SW_Push, Button_Switch_THT:SW_PUSH_6mm_H4.3mm, F.Cu at (40.1, 104.5)
- added SW3: MFP 113 D, Button_Switch_THT:SW_Slide_1P2T_CK_OS102011MS2Q, F.Cu at (42.0, 99.6)
- added U5: PC817, Package_DIP:DIP-4_W8.89mm_SMDSocket_LongPads, F.Cu at (44.8, 86.7)
- C10, C11: value 100n -> 10n
- C12, C13: value 100n -> 10u
- C14: value 22u -> 100n
- C15: value 22u/25V -> 100n
- C8: value 22u -> 10u
- D1: value LED-GR -> GR
- D2: value LED-YEL -> YEL
- D3: value LED-RED -> RED
- D4: value LED-BLUE -> BLUE
- D5: value 1N4007 -> 1N5819
- D6: value LED-BLUE -> 1N5819; footprint LED_SMD:LED_0805_2012Metric -> Diode_SMD:D_SOD-123
- D8: value SM712_SOT23 -> GR; footprint Package_TO_SOT_SMD:SOT-23 -> LED_SMD:LED_0805_2012Metric
- J6, J7: value Screw_Terminal_01x02 -> MV132
- R10: value 1k -> 2k2
- R11: value 0.1R -> 2k2; footprint Resistor_SMD:R_1206_3216Metric -> Resistor_SMD:R_0805_2012Metric
- R12, R13, R14: value 10k -> 1k
- R15: value 220R -> 10k
- R18: value 10M -> 10k; footprint Resistor_THT:R_Axial_DIN0207_L6.3mm_D2.5mm_P10.16mm_Horizontal -> Resistor_SMD:R_0805_2012Metric
- U3: value ADM2483xRW -> PC817; footprint Package_SO:SOIC-16W_7.5x10.3mm_P1.27mm -> Package_DIP:DIP-4_W8.89mm_SMDSocket_LongPads
- U4: value ADUM1250 -> PC817; footprint Package_SO:SO-8_3.9x4.9mm_P1.27mm -> Package_DIP:DIP-4_W8.89mm_SMDSocket_LongPads
- U6: value LM78M05_TO252 -> PC817; footprint Package_TO_SOT_SMD:TO-252-2 -> Package_DIP:DIP-4_W8.89mm_SMDSocket_LongPads
- U7: value INA219AxDCN -> 74HC123; footprint Package_TO_SOT_SMD:SOT-23-8 -> Package_SO:SOIC-16_3.9x9.9mm_P1.27mm
- moved J7 120.5 mm to (64.6, 52.1)
- moved J5 118.9 mm to (56.1, 50.3)
- moved J4 118.3 mm to (39.5, 52.9)
- moved J6 114.0 mm to (79.5, 52.6)
- moved D5 107.0 mm to (76.5, 159.9)
- moved R10 104.8 mm to (74.1, 104.9)
- moved D6 104.0 mm to (75.5, 93.7)
- moved C15 103.4 mm to (73.1, 154.1)
- moved C14 102.1 mm to (73.9, 140.1)
- moved C16 100.4 mm to (71.5, 166.3)
- moved U3 98.6 mm to (85.7, 180.7)
- moved R14 98.0 mm to (74.1, 172.1)
- moved R15 95.5 mm to (70.7, 142.5)
- moved R16 94.6 mm to (78.5, 165.7)
- moved U6 93.8 mm to (84.9, 147.7)
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Connections:
- net BOOT0 renamed /BOOT
- net LED_BLUE renamed /LED_BLUE
- net LED_GR renamed /LED_GR
- net LED_RED renamed /LED_RED
- net LED_YEL renamed /LED_YEL
- C10 pad 1: GND -> Net-(C10-Pad1)
- C10 pad 2: +3V3 -> Net-(C10-Pad2)
- C11 pad 1: GND -> Net-(C11-Pad1)
- C11 pad 2: +3V3 -> Net-(C11-Pad2)
- C12 pad 1: +5VA -> +5V
- C12 pad 2: GNDA -> GND
- C13 pad 1: GNDA -> +5V
- C13 pad 2: ADM_IN- -> GND
- C14 pad 1: GNDA -> Net-(C14-Pad1)
- C14 pad 2: +5VA -> GND
- C15 pad 1: GNDA -> +3V3
- C15 pad 2: Net-(C15-Pad2) -> GND
- C16 pad 1: +5VA -> Net-(C16-Pad1)
- C16 pad 2: GNDA -> GND
- D5 pad 1: Net-(C15-Pad2) -> Net-(C10-Pad1)
- D5 pad 2: +12VA -> /DCC cutting/J1
- D6 pad 1: GNDA -> /DCC cutting/J1
- D6 pad 2: Net-(D6-Pad2) -> Net-(C10-Pad2)
- D8 pad 1: /MTB-BUS+ -> Net-(C10-Pad2)
- D8 pad 2: /MTB-BUS- -> Net-(D8-Pad2)
- J4 pad 1: +12VA -> /DCC cutting/J1
- J4 pad 2: GNDA -> /DCC cutting/TW2
- J4 pad 3: /MTB-BUS+ -> /DCC cutting/TW3
- J4 pad 4: /MTB-BUS- -> /DCC cutting/TW4
- J4 pad 5: GNDA -> /DCC cutting/TW5
- J4 pad 6: +12VA -> /DCC cutting/K1
- J5 pad 1: +12VA -> /DCC cutting/J2
- J5 pad 2: GNDA -> /DCC cutting/TW2
- J5 pad 3: /MTB-BUS+ -> /DCC cutting/TW3
- J5 pad 4: /MTB-BUS- -> /DCC cutting/TW4
- J5 pad 5: GNDA -> /DCC cutting/TW5
- J5 pad 6: +12VA -> /DCC cutting/K2
- J6 pad 1: GNDA -> /DCC cutting/J1
- J6 pad 2: +12VA -> /DCC cutting/K1
- J7 pad 1: /MTB-BUS- -> /DCC cutting/J2
- J7 pad 2: /MTB-BUS+ -> /DCC cutting/K2
- R10 pad 1: Net-(D6-Pad2) -> Net-(D8-Pad2)
- R10 pad 2: +5VA -> Net-(R10-Pad2)
- R11 pad 1: ADM_IN- -> Net-(D9-Pad2)
- R11 pad 2: +5VA -> Net-(R11-Pad2)
- R12 pad 1: +5VA -> Net-(Q1-Pad1)
- R12 pad 2: /MTB-BUS+ -> /DCC cutting/REL1CTRL
- R13 pad 1: /MTB-BUS- -> Net-(Q2-Pad1)
- R13 pad 2: GNDA -> /DCC cutting/REL2CTRL
- R14 pad 1: Net-(R14-Pad1) -> /DCC cutting/REL1CTRL
- R14 pad 2: +5VA -> Net-(D12-Pad2)
- R15 pad 1: /MTB-BUS- -> /DCC cutting/REL1CTRL
- R15 pad 2: /MTB-BUS+ -> GND
- R16 pad 1: Net-(R16-Pad1) -> /SW_GO
- R16 pad 2: +5VA -> +3V3
- R18 pad 1: GNDA -> /SW_STOP
- R18 pad 2: GND -> +3V3
- R8 pad 1: I2C_SCL -> Net-(R29-Pad2)
- R9 pad 1: I2C_SDA -> Net-(R30-Pad1)
- U1 pad 18: unconnected-(U1-Pad18) -> /IO1DCC
- U1 pad 19: unconnected-(U1-Pad19) -> /IO2DCC
- U1 pad 20: USART_MTB_DIR -> /REL1CTRL
- U1 pad 21: USART_MTB_TX -> /LED_STOP
- U1 pad 22: USART_MTB_RX -> /LED_GO
- U1 pad 39: unconnected-(U1-Pad39) -> /REL2CTRL
- U1 pad 41: unconnected-(U1-Pad41) -> OUT_ALERT
- U1 pad 42: unconnected-(U1-Pad42) -> OUT_ON
- U1 pad 43: unconnected-(U1-Pad43) -> /SW_GO
- U1 pad 45: I2C_SCL -> /SW_STOP
- U1 pad 46: I2C_SDA -> /SW_OVERRIDE
- U1 pad 8: unconnected-(U1-Pad8) -> GND
- U3 pad 1: +3V3 -> Net-(R23-Pad2)
- U3 pad 3: USART_MTB_RX -> Net-(J9-Pad2)
- U3 pad 4: USART_MTB_DIR -> Net-(J9-Pad1)
- U4 pad 1: +3V3 -> Net-(R24-Pad2)
- U4 pad 2: I2C_SDA -> GND
- U4 pad 3: I2C_SCL -> Net-(J10-Pad2)
- U4 pad 4: GND -> Net-(J10-Pad1)
- U6 pad 1: Net-(C15-Pad2) -> Net-(C11-Pad2)
- U6 pad 2: GNDA -> Net-(R11-Pad2)
- U6 pad 3: Net-(JP6-Pad2) -> GND
- U7 pad 1: +5VA -> GND
- U7 pad 2: ADM_IN- -> /REL1CTRL
- U7 pad 3: GNDA -> +3V3
- U7 pad 4: +5VA -> unconnected-(U7-Pad4)
- U7 pad 5: Net-(R16-Pad1) -> /DCC cutting/REL2CTRL
- U7 pad 6: Net-(R14-Pad1) -> GND
- U7 pad 7: GNDA -> Net-(C16-Pad1)
- U7 pad 8: GNDA -> GND
Routing:
- net +5VA: track 107.9 -> 0.00 mm, vias 5 -> 0
- net /MTB-BUS-: track 79.1 -> 0.00 mm, vias 2 -> 0
- net /MTB-BUS+: track 75.0 -> 0.00 mm, vias 3 -> 0
- net +3V3: track 179.2 -> 110.6 mm, vias 10 -> 5
- net +12VA: track 60.6 -> 0.00 mm
- net I2C_SDA: track 50.7 -> 0.00 mm, vias 4 -> 0
- net I2C_SCL: track 48.6 -> 0.00 mm, vias 4 -> 0
- net +5V: track 124.0 -> 76.9 mm
- net ADM_IN-: track 31.5 -> 0.00 mm, vias 2 -> 0
- net USART_MTB_TX: track 21.7 -> 0.00 mm
- net USART_MTB_DIR: track 21.1 -> 0.00 mm, vias 2 -> 0
- net USART_MTB_RX: track 18.1 -> 0.00 mm
- net Net-(R14-Pad1): track 13.9 -> 0.00 mm, vias 2 -> 0
- net Net-(D6-Pad2): track 10.6 -> 0.00 mm
- net Net-(JP7-Pad3): track 10.6 -> 0.00 mm
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- removed copper zone on B.Cu, net GNDA
- removed copper zone on F.Cu, net GNDA

Commit message: Draw & route part of PCB.
Parts:
- D10, D11: footprint Diode_THT:D_DO-35_SOD27_P7.62mm_Horizontal -> Diode_SMD:D_0805_2012Metric_Pad1.15x1.40mm_HandSolder
- moved R14 139.2 mm to (124.6, 42.4)
- moved D14 134.0 mm to (173.7, 124.7), turned to 90 degrees
- moved SW3 128.8 mm to (168.4, 124.7), turned to 180 degrees
- moved D9 127.6 mm to (174.8, 50.8), turned to 90 degrees
- moved R30 126.2 mm to (166.4, 87.9), turned to 90 degrees
- moved U3 115.9 mm to (105.7, 66.5), turned to 90 degrees
- moved R11 115.8 mm to (174.2, 70.9), turned to -90 degrees
- moved R25 114.5 mm to (159.0, 85.1)
- moved D22 114.0 mm to (166.1, 65.3)
- moved D18 113.9 mm to (166.1, 62.5)
- moved R20 113.4 mm to (173.7, 113.8), turned to 90 degrees
- moved D16 112.9 mm to (157.2, 125.0), turned to 90 degrees
- moved SW2 111.9 mm to (149.4, 128.2), turned to 90 degrees
- moved D5 111.3 mm to (127.3, 61.0), turned to 0 degrees
- moved U4 110.6 mm to (112.8, 66.5), turned to 90 degrees
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Connections:
- D7 pad 4: USBD+ -> USBD-
- D7 pad 6: USBD- -> USBD+
Routing:
- net +3V3: track 110.6 -> 27.0 mm, vias 5 -> 17
- net /DCC cutting/K1: track 0.00 -> 39.8 mm
- net /DCC cutting/J1: track 0.00 -> 33.8 mm
- net /LED_GR: track 32.6 -> 0.00 mm
- net Net-(D17-Pad1): track 0.00 -> 29.5 mm, vias 0 -> 2
- net /LED_YEL: track 28.6 -> 0.00 mm
- net /LED_BLUE: track 28.2 -> 0.00 mm
- net DBG_CTS: track 28.0 -> 0.00 mm, vias 1 -> 0
- net Net-(J8-Pad2): track 27.1 -> 0.00 mm
- net /LED_RED: track 26.7 -> 0.00 mm
- net +5V: track 76.9 -> 50.2 mm, vias 3 -> 11
- net Net-(J8-Pad1): track 25.4 -> 0.00 mm
- net /BOOT: track 24.8 -> 0.00 mm, vias 2 -> 0
- net Net-(D21-Pad1): track 0.00 -> 24.7 mm, vias 0 -> 1
- net RST: track 32.6 -> 8.12 mm, vias 1 -> 0
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- added copper zone on F.Cu, net +3V3
- added copper zone on In1.Cu, net +3V3
- added copper zone on F.Cu, net +5V
- added copper zone on In2.Cu, net GND
Other:
- copper layers 2 -> 4

Commit message: Route another part of PCB.
Parts:
- moved R28 42.2 mm to (126.7, 99.8)
- moved C16 41.5 mm to (131.1, 99.8), turned to 0 degrees
- moved R27 40.0 mm to (128.0, 89.2), turned to 180 degrees
- moved U7 38.3 mm to (127.8, 94.5), turned to 90 degrees
- moved C14 34.4 mm to (123.7, 89.2), turned to 180 degrees
- moved C15 31.7 mm to (120.9, 94.5), turned to -90 degrees
- moved C10 27.2 mm to (146.3, 70.9), turned to 90 degrees
- moved JP3 27.0 mm to (170.4, 88.6), turned to -90 degrees
- moved R19 24.3 mm to (164.3, 113.8), turned to 90 degrees
- moved TP6 23.6 mm to (104.9, 91.7)
- moved R8 23.5 mm to (149.1, 79.0), turned to -90 degrees
- moved R10 22.5 mm to (136.7, 70.9)
- moved D10 22.1 mm to (124.0, 81.3), turned to 90 degrees
- moved R14 21.5 mm to (116.8, 62.5), turned to 90 degrees
- moved R29 20.9 mm to (146.6, 79.0), turned to 90 degrees
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Routing:
- net /DCC cutting/REL2CTRL: track 2.75 -> 69.5 mm, vias 0 -> 3
- net Net-(C10-Pad2): track 0.00 -> 49.1 mm, vias 0 -> 2
- net /SW_OVERRIDE: track 0.00 -> 46.3 mm
- net /DCC cutting/REL1CTRL: track 0.00 -> 38.5 mm, vias 0 -> 2
- net Net-(K1-Pad7): track 0.00 -> 34.8 mm
- net Net-(K1-Pad4): track 0.00 -> 32.5 mm
- net GND: track 4.43 -> 34.1 mm, vias 35 -> 44
- net Net-(D8-Pad2): track 0.00 -> 29.1 mm, vias 0 -> 2
- net +3V3: track 27.0 -> 53.9 mm, vias 17 -> 26
- net /SW_STOP: track 0.00 -> 25.9 mm
- net /SW_GO: track 0.00 -> 24.4 mm
- net +5V: track 50.2 -> 69.6 mm, vias 11 -> 12
- net /DCC cutting/K1: track 39.8 -> 55.9 mm, vias 0 -> 1
- net Net-(D12-Pad2): track 0.00 -> 15.4 mm
- net /DCC cutting/J1: track 33.8 -> 48.9 mm
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
Commit message: Wire everything.
Parts:
- moved JP3 43.4 mm to (132.7, 110.1), turned to 180 degrees
- moved JP2 38.0 mm to (148.9, 85.0), turned to 0 degrees
- moved J3 30.7 mm to (161.3, 88.6), turned to -90 degrees
- moved JP4 22.7 mm to (161.8, 110.0), turned to 0 degrees
- moved JP1 19.8 mm to (161.8, 107.4), turned to 0 degrees
- moved J8 2.56 mm to (167.9, 93.9), turned to 90 degrees
- moved C5 0.08 mm to (150.6, 110.3)
Routing:
- net OUT_ALERT: track 0.00 -> 52.5 mm, vias 0 -> 2
- net OUT_ON: track 0.00 -> 49.2 mm, vias 0 -> 2
- net /IO2DCC: track 0.00 -> 40.9 mm, vias 0 -> 2
- net Net-(J8-Pad2): track 0.00 -> 34.4 mm, vias 0 -> 1
- net SWDIO: track 0.00 -> 32.0 mm, vias 0 -> 1
- net Net-(J8-Pad1): track 0.00 -> 31.9 mm, vias 0 -> 1
- net SWCLK: track 0.00 -> 31.3 mm, vias 0 -> 1
- net /LED_BLUE: track 0.00 -> 29.7 mm, vias 0 -> 2
- net /LED_RED: track 0.00 -> 26.3 mm
- net /REL2CTRL: track 0.00 -> 24.9 mm
- net /REL1CTRL: track 0.00 -> 24.4 mm, vias 0 -> 2
- net /LED_GO: track 0.00 -> 23.2 mm, vias 0 -> 2
- net /LED_YEL: track 0.00 -> 23.2 mm
- net /LED_STOP: track 0.00 -> 22.8 mm, vias 0 -> 2
- net /LED_GR: track 0.00 -> 20.6 mm
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- added copper zone on In1.Cu, net +5V

Commit message: Silkscreen.
Parts:
- moved TP6 14.2 mm to (117.6, 85.3)
- moved H2 2.81 mm to (166.4, 57.4)
- moved JP2 0.54 mm to (148.3, 85.0)
Routing:
- net Net-(J3-Pad4): track 7.11 -> 8.01 mm
- net GND: vias 52 -> 53
Other:
- board text added: "DC-01 v1.0"
- board text added: "KMŽ Brno I Jan Horáček 2023"
- board text removed: "+12V"
- board text removed: "+R"
- board text removed: "-R"
- board text removed: "BL"
- board text removed: "GR"
- board text removed: "JLCJLCJLCJLC"
- board text removed: "KMŽ Brno I Jan Horáček 2022"
- board text removed: "MTB-USB v4.3"
- board text removed: "MTBbus"
- board text removed: "PROG conn pinout"
- board text removed: "RED"
- board text removed: "YEL"

Commit message: Tweak tracks width, silkscreen, GND vias.
Parts:
- moved F1 1.37 mm to (153.7, 61.2), turned to 180 degrees
- moved F2 1.37 mm to (159.8, 61.2), turned to 0 degrees
Routing:
- net /DCC cutting/J2: track 23.0 -> 27.6 mm
- net /DCC cutting/K2: track 21.2 -> 22.9 mm
- net Net-(D17-Pad1): track 29.4 -> 28.6 mm
- net +3V3: track 62.9 -> 63.4 mm
- net GND: vias 53 -> 69

Commit message: Fix DRC errors.
Routing:
- net Net-(J9-Pad2): track 21.5 -> 20.9 mm
- net Net-(J9-Pad1): track 21.2 -> 20.5 mm
- net Net-(J10-Pad1): track 21.5 -> 20.8 mm
- net Net-(J10-Pad2): track 21.9 -> 21.2 mm
Other:
- board text removed: "A"
- board text removed: "B"
Changed lines of the file:
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@@
     (effects (font (size 2 2) (thickness 0.15)))
-  )
-  (gr_text "A" (at 106.934 70.358) (layer "F.SilkS")
-    (effects (font (size 1 1) (thickness 0.15)))
   )
   (gr_text "VCC" (at 153.67 91.694 90) (layer "F.SilkS")
@@
   )
   (gr_text "3V3" (at 163.576 102.87) (layer "F.SilkS")
-    (effects (font (size 1 1) (thickness 0.15)))
-  )
-  (gr_text "B" (at 104.394 70.358) (layer "F.SilkS")
     (effects (font (size 1 1) (thickness 0.15)))
   )
@@
   (segment (start 119.126 50.8) (end 118.618 51.308) (width 0.3) (layer "In2.Cu") (net 2))
   (segment (start 118.618 51.308) (end 118.618 77.216) (width 0.3) (layer "In2.Cu") (net 2))
-  (segment (start 109.536 102.63) (end 109.55 102.616) (width 0.7) (layer "F.Cu") (net 3))
-  (segment (start 150.6235 109.156) (end 150.5575 109.156) (width 0.3) (layer "F.Cu") (net 3))
   (segment (start 149.098 102.14) (end 150.2075 102.14) (width 0.3) (layer "F.Cu") (net 3))
   (segment (start 150.5575 109.156) (end 149.62575 108.22425) (width 0.3) (layer "F.Cu") (net 3))
@@
   (segment (start 150.836 104.14) (end 152.042 105.346) (width 0.3) (layer "F.Cu") (net 4))
   (segment (start 149.098 104.14) (end 150.836 104.14) (width 0.3) (layer "F.Cu") (net 4))
-  (segment (start 154.178 105.4105) (end 154.1135 105.346) (width 0.3) (layer "F.Cu") (net 4))
   (segment (start 153.228 108.458) (end 153.228 106.2315) (width 0.3) (layer "F.Cu") (net 4))
   (segment (start 149.098 103.64) (end 152.1195 103.64) (width 0.3) (layer "F.Cu") (net 5))
@@
   (segment (start 102.87 59.69) (end 103.914 58.646) (width 0.6) (layer "F.Cu") (net 70))
   (segment (start 103.914 58.646) (end 103.914 50.7) (width 0.6) (layer "F.Cu") (net 70))
-  (segment (start 104.394 51.18) (end 103.914 50.7) (width 0.4) (layer "F.Cu") (net 70))
   (segment (start 105.41 57.658) (end 107.414 55.654) (width 0.6) (layer "F.Cu") (net 71))
   (segment (start 107.414 55.654) (end 107.414 50.7) (width 0.6) (layer "F.Cu") (net 71))
   (segment (start 105.41 70.739) (end 105.41 57.658) (width 0.6) (layer "F.Cu") (net 71))
-  (segment (start 106.934 51.18) (end 107.414 50.7) (width 0.4) (layer "F.Cu") (net 71))
   (segment (start 109.22 57.658) (end 111.026 55.852) (width 0.6) (layer "F.Cu") (net 72))
   (segment (start 109.22 70.739) (end 109.22 57.658) (width 0.6) (layer "F.Cu") (net 72))
   (segment (start 111.026 55.852) (end 111.026 50.7) (width 0.6) (layer "F.Cu") (net 72))
-  (segment (start 111.506 51.18) (end 111.026 50.7) (width 0.4) (layer "F.Cu") (net 72))
-  (segment (start 114.046 51.18) (end 114.526 50.7) (width 0.4) (layer "F.Cu") (net 73))
   (segment (start 111.76 58.166) (end 114.526 55.4) (width 0.6) (layer "F.Cu") (net 73))
   (segment (start 111.76 70.739) (end 111.76 58.166) (width 0.6) (layer "F.Cu") (net 73))

Commit message: Minor silkscreen tweaks.
Parts:
- removed TP6: TestPoint, TestPoint:TestPoint_Loop_D3.50mm_Drill1.4mm_Beaded
- added REF**: OSHW-Logo2_9.8x8mm_SilkScreen, Symbol:OSHW-Logo2_9.8x8mm_SilkScreen, F.Cu at (123.7, 105.7)
- added TP1: TestPoint, TestPoint:TestPoint_Loop_D3.50mm_Drill1.4mm_Beaded, F.Cu at (117.6, 85.3)
