File: pcb/dc01.kicad_pcb (KiCad board)
At the start: 4 copper layers, 76 x 84 mm, 104 parts, among them J1 USB_C_Receptacle_USB2.0, J10 MV132, J2 PROG/DEBUG, J3 Conn_01x06, J4 RJ12, J5 RJ12, J6 MV132, J7 MV132, J8 Conn_01x02, J9 MV132, K1 AZ850-5, K2 AZ850-5, Q1 2N7002, Q2 2N7002, SW1 SW_Push, SW2 SW_Push, SW3 MFP 113 D, U1 STM32F103C8Tx, U2 AMS1117-3.3, U3 PC817, U4 PC817, U5 PC817, U6 PC817, U7 74HC123, Y1 8 MHz

Commit message: Do not use 2 different types of diodes.
Parts:
- D10, D11: footprint Diode_SMD:D_0805_2012Metric_Pad1.15x1.40mm_HandSolder -> Diode_SMD:D_SOD-123
Routing:
- net +5V: track 77.5 -> 78.0 mm

Commit message: Tweak silkscreen.
Parts:
- added REF**: WEEE-Logo_8.4x12mm_SilkScreen, Symbol:WEEE-Logo_8.4x12mm_SilkScreen, B.Cu at (110.5, 68.3)
Other:
- board text added: "https://www.kmz-brno.cz/ https://github.com/kmzbrnoI/dc01"

Commit message: Add pull-down resistors to relay logic signals.
Parts:
- added R31: 10k, Resistor_SMD:R_0805_2012Metric, F.Cu at (140.3, 93.7)
- added R32: 10k, Resistor_SMD:R_0805_2012Metric, F.Cu at (136.4, 93.7)
- D10, D11: value 1N4148 -> 1N5819
Routing:
- net /REL1CTRL: track 24.4 -> 26.4 mm
- net /REL2CTRL: track 24.9 -> 26.5 mm
Other:
- board text added: "DC-01 v1.1"
- board text removed: "DC-01 v1.0"
Changed lines of the file:
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@@
     (descr "SOIC, 16 Pin (JEDEC MS-012AC, https://www.analog.com/media/en/package-pcb-resources/package/pkg_pdf/soic_narrow-r/r_16.pdf), generated with kicad-footprint-generator ipc_gullwing_generator.py")
     (tags "SOIC SO")
+    (property "JLCPCB_CORRECTION" "0;0;270")
     (property "LCSC" "C91435")
     (property "Sheetfile" "safesig.kicad_sch")
@@
     (property "Sheetname" "")
     (attr smd)
-    (fp_text reference "C6" (at 0 -1.818) (layer "F.SilkS")
+    (fp_text reference "C6" (at -3.429 0.087) (layer "F.SilkS")
       (effects (font (size 1 1) (thickness 0.15)))
     )
@@
       (effects (font (size 1 1) (thickness 0.15)))
     )
-    (fp_text value "1N4148" (at 0 2.1 90) (layer "F.Fab")
+    (fp_text value "1N5819" (at 0 2.1 90) (layer "F.Fab")
       (effects (font (size 1 1) (thickness 0.15)))
     )
@@
     )
   )
+  (footprint "Resistor_SMD:R_0805_2012Metric" (layer "F.Cu")
+    (at 136.4215 93.726 180)
+    (descr "Resistor SMD 0805 (2012 Metric), square (rectangular) end terminal, IPC_7351 nominal, (Body size source: IPC-SM-782 page 72, https://www.pcb-3d.com/wordpress/wp-content/uploads/ipc-sm-782a_amendment_1_and_2.pdf), generated with kicad-footprint-generator")
+    (tags "resistor")
+    (property "LCSC" "C17414")
+    (property "Sheetfile" "safesig.kicad_sch")
+    (property "Sheetname" "Safe relay signal generation")
+    (attr smd)
+    (fp_text reference "R32" (at 0 -1.65) (layer "F.SilkS")
+      (effects (font (size 1 1) (thickness 0.15)))
+    )
+    (fp_text value "10k" (at 0 1.65) (layer "F.Fab")
+      (effects (font (size 1 1) (thickness 0.15)))
+    )
+    (fp_text user "${REFERENCE}" (at 0 0) (layer "F.Fab")
+      (effects (font (size 0.5 0.5) (thickness 0.08)))
+    )
+    (fp_line (start -0.227064 -0.735) (end 0.227064 -0.735) (layer "F.SilkS") (width 0.12))
+    (fp_line (start -0.227064 0.735) (end 0.227064 0.735) (layer "F.SilkS") (width 0.12))
+    (fp_line (start -1.68 -0.95) (end 1.68 -0.95) (layer "F.CrtYd") (width 0.05))
+    (fp_line (start 1.68 0.95) (end -1.68 0.95) (layer "F.CrtYd") (width 0.05))
+    (fp_line (start -1.68 0.95) (end -1.68 -0.95) (layer "F.CrtYd") (width 0.05))
+    (fp_line (start 1.68 -0.95) (end 1.68 0.95) (layer "F.CrtYd") (width 0.05))
+    (fp_line (start 1 0.625) (end -1 0.625) (layer "F.Fab") (width 0.1))
+    (fp_line (start -1 0.625) (end -1 -0.625) (layer "F.Fab") (width 0.1))
+    (fp_line (start 1 -0.625) (end 1 0.625) (layer "F.Fab") (width 0.1))
+    (fp_line (start -1 -0.625) (end 1 -0.625) (layer "F.Fab") (width 0.1))
+    (pad "1" smd roundrect (at -0.9125 0 180) (size 1.025 1.4) (layers "F.Cu" "F.Paste" "F.Mask") (roundrect_rratio 0.243902)
+      (net 2 "GND") (pintype "passive"))
+    (pad "2" smd roundrect (at 0.9125 0 180) (size 1.025 1.4) (layers "F.Cu" "F.Paste" "F.Mask") (roundrect_rratio 0.243902)
+      (net 105 "/REL2CTRL") (pintype "passive"))
+    (model "${KICAD6_3DMODEL_DIR}/Resistor_SMD.3dshapes/R_0805_2012Metric.wrl"
+      (offset (xyz 0 0 0))
+      (scale (xyz 1 1 1))
+      (rotate (xyz 0 0 0))
+    )
+  )
   (footprint "LED_SMD:LED_0805_2012Metric" (layer "F.Cu")
     (at 119.126 52.832 -90)
@@
       (effects (font (size 1 1) (thickness 0.15)))
     )
-    (fp_text value "1N4148" (at 0 2.1 90) (layer "F.Fab")
+    (fp_text value "1N5819" (at 0 2.1 90) (layer "F.Fab")
       (effects (font (size 1 1) (thickness 0.15)))
     )
@@
     )
   )
+  (footprint "Resistor_SMD:R_0805_2012Metric" (layer "F.Cu")
+    (at 140.335 93.726)
+    (descr "Resistor SMD 0805 (2012 Metric), square (rectangular) end terminal, IPC_7351 nominal, (Body size source: IPC-SM-782 page 72, https://www.pcb-3d.com/wordpress/wp-content/uploads/ipc-sm-782a_amendment_1_and_2.pdf), generated with kicad-footprint-generator")
+    (tags "resistor")
+    (property "LCSC" "C17414")
+    (property "Sheetfile" "safesig.kicad_sch")
+    (property "Sheetname" "Safe relay signal generation")
+    (attr smd)
+    (fp_text reference "R31" (at 0 1.651) (layer "F.SilkS")
+      (effects (font (size 1 1) (thickness 0.15)))
+    )
+    (fp_text value "10k" (at 0 1.65) (layer "F.Fab")
+      (effects (font (size 1 1) (thickness 0.15)))
+    )
+    (fp_text user "${REFERENCE}" (at 0 0) (layer "F.Fab")
+      (effects (font (size 0.5 0.5) (thickness 0.08)))
+    )
+    (fp_line (start -0.227064 -0.735) (end 0.227064 -0.735) (layer "F.SilkS") (width 0.12))
+    (fp_line (start -0.227064 0.735) (end 0.227064 0.735) (layer "F.SilkS") (width 0.12))
+    (fp_line (start 1.68 -0.95) (end 1.68 0.95) (layer "F.CrtYd") (width 0.05))
+    (fp_line (start 1.68 0.95) (end -1.68 0.95) (layer "F.CrtYd") (width 0.05))
+    (fp_line (start -1.68 0.95) (end -1.68 -0.95) (layer "F.CrtYd") (width 0.05))
+    (fp_line (start -1.68 -0.95) (end 1.68 -0.95) (layer "F.CrtYd") (width 0.05))
+    (fp_line (start -1 -0.625) (end 1 -0.625) (layer "F.Fab") (width 0.1))
+    (fp_line (start -1 0.625) (end -1 -0.625) (layer "F.Fab") (width 0.1))
+    (fp_line (start 1 0.625) (end -1 0.625) (layer "F.Fab") (width 0.1))
+    (fp_line (start 1 -0.625) (end 1 0.625) (layer "F.Fab") (width 0.1))
+    (pad "1" smd roundrect (at -0.9125 0) (size 1.025 1.4) (layers "F.Cu" "F.Paste" "F.Mask") (roundrect_rratio 0.243902)
+      (net 2 "GND") (pintype "passive"))
+    (pad "2" smd roundrect (at 0.9125 0) (size 1.025 1.4) (layers "F.Cu" "F.Paste" "F.Mask") (roundrect_rratio 0.243902)
+      (net 104 "/REL1CTRL") (pintype "passive"))
+    (model "${KICAD6_3DMODEL_DIR}/Resistor_SMD.3dshapes/R_0805_2012Metric.wrl"
+      (offset (xyz 0 0 0))
+      (scale (xyz 1 1 1))
+      (rotate (xyz 0 0 0))
+    )
+  )
   (footprint "TerminalBlock_4Ucon:TerminalBlock_4Ucon_1x02_P3.50mm_Horizontal" (layer "F.Cu")
     (at 103.914 50.7)
@@
     (effects (font (size 1.5 1.5) (thickness 0.15)))
   )
-  (gr_text "DC-01\nv1.0" (at 107.442 64.008) (layer "F.SilkS")
+  (gr_text "DC-01\nv1.1" (at 107.442 64.008) (layer "F.SilkS")
     (effects (font (size 2 2) (thickness 0.2)))
   )
@@
   (segment (start 136.278 95.548) (end 141.778 95.548) (width 0.3) (layer "F.Cu") (net 104))
   (segment (start 124.578 96.954) (end 124.587 96.963) (width 0.3) (layer "F.Cu") (net 104))
+  (segment (start 141.778 94.2565) (end 141.2475 93.726) (width 0.3) (layer "F.Cu") (net 104))
   (segment (start 141.778 95.548) (end 144.1855 97.9555) (width 0.3) (layer "F.Cu") (net 104))
+  (segment (start 141.778 95.548) (end 141.778 94.2565) (width 0.3) (layer "F.Cu") (net 104))
   (segment (start 124.578 94.848) (end 124.578 96.954) (width 0.3) (layer "F.Cu") (net 104))
   (via (at 136.278 95.548) (size 0.7) (drill 0.4) (layers "F.Cu" "B.Cu") (net 104))
@@
   (segment (start 136.178 95.448) (end 124.978 95.448) (width 0.3) (layer "B.Cu") (net 104))
   (segment (start 136.278 95.548) (end 136.178 95.448) (width 0.3) (layer "B.Cu") (net 104))
-  (segment (start 132.078 94.448) (end 130.937 93.307) (width 0.3) (layer "F.Cu") (net 105))
-  (segment (start 133.978 94.448) (end 132.078 94.448) (width 0.3) (layer "F.Cu") (net 105))
-  (segment (start 143.478 106.148) (end 143.478 101.858541) (width 0.3) (layer "F.Cu") (net 105))
   (segment (start 140.867459 99.248) (end 135.878 99.248) (width 0.3) (layer "F.Cu") (net 105))
-  (segment (start 135.178 98.548) (end 135.178 95.648) (width 0.3) (layer "F.Cu") (net 105))
-  (segment (start 143.1855 107.5525) (end 143.1855 106.4405) (width 0.3) (layer "F.Cu") (net 105))
-  (segment (start 143.478 101.858541) (end 140.867459 99.248) (width 0.3) (layer "F.Cu") (net 105))
-  (segment (start 130.937 93.307) (end 130.937 92.013) (width 0.3) (layer "F.Cu") (net 105))
   (segment (start 135.878 99.248) (end 135.178 98.548) (width 0.3) (layer "F.Cu") (net 105))
+  (segment (start 135.178 98.548) (end 135.178 94.057) (width 0.3) (layer "F.Cu") (net 105))
   (segment (start 143.1855 106.4405) (end 143.478 106.148) (width 0.3) (layer "F.Cu") (net 105))
-  (segment (start 135.178 95.648) (end 133.978 94.448) (width 0.3) (layer "F.Cu") (net 105))
+  (segment (start 135.509 93.726) (end 131.356 93.726) (width 0.3) (layer "F.Cu") (net 105))
+  (segment (start 131.356 93.726) (end 130.937 93.307) (width 0.3) (layer "F.Cu") (net 105))
+  (segment (start 130.937 93.307) (end 130.937 92.013) (width 0.3) (layer "F.Cu") (net 105))
+  (segment (start 143.1855 107.5525) (end 143.1855 106.4405) (width 0.3) (layer "F.Cu") (net 105))
+  (segment (start 143.478 106.148) (end 143.478 101.858541) (width 0.3) (layer "F.Cu") (net 105))
+  (segment (start 135.178 94.057) (end 135.509 93.726) (width 0.3) (layer "F.Cu") (net 105))
+  (segment (start 143.478 101.858541) (end 140.867459 99.248) (width 0.3) (layer "F.Cu") (net 105))
   (zone (net 2) (net_name "GND") (layer "F.Cu") (hatch edge 0.508)
     (connect_pads (clearance 0.3))

Commit message: Add separate resistors for LEDs.
Parts:
- added R33: 22k, Resistor_SMD:R_0805_2012Metric, F.Cu at (164.5, 33.7)
- added R34: 22k, Resistor_SMD:R_0805_2012Metric, F.Cu at (171.7, 67.7)
Connections:
- R10 pad 1: Net-(D8-Pad2) -> Net-(C10-Pad2)
- R11 pad 1: Net-(D9-Pad2) -> Net-(C11-Pad1)
Routing:
- net Net-(C11-Pad1): track 22.3 -> 28.7 mm, vias 0 -> 2
- net Net-(C11-Pad2): track 13.7 -> 17.9 mm
- net Net-(D9-Pad2): track 22.2 -> 21.6 mm
Changed lines of the file:
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@@
     (fp_line (start 1 -0.625) (end 1 0.625) (layer "F.Fab") (width 0.1))
     (pad "1" smd roundrect (at -0.9125 0 270) (size 1.025 1.4) (layers "F.Cu" "F.Paste" "F.Mask") (roundrect_rratio 0.243902)
-      (net 32 "Net-(D9-Pad2)") (pintype "passive"))
+      (net 13 "Net-(C11-Pad1)") (pintype "passive"))
     (pad "2" smd roundrect (at 0.9125 0 270) (size 1.025 1.4) (layers "F.Cu" "F.Paste" "F.Mask") (roundrect_rratio 0.243902)
       (net 90 "Net-(R11-Pad2)") (pintype "passive"))
@@
     (fp_line (start -1 -0.625) (end 1 -0.625) (layer "F.Fab") (width 0.1))
     (pad "1" smd roundrect (at -0.9125 0 270) (size 1.025 1.4) (layers "F.Cu" "F.Paste" "F.Mask") (roundrect_rratio 0.243902)
-      (net 31 "Net-(D8-Pad2)") (pintype "passive"))
+      (net 8 "Net-(C10-Pad2)") (pintype "passive"))
     (pad "2" smd roundrect (at 0.9125 0 270) (size 1.025 1.4) (layers "F.Cu" "F.Paste" "F.Mask") (roundrect_rratio 0.243902)
       (net 89 "Net-(R10-Pad2)") (pintype "passive"))
@@
   )
   (footprint "Resistor_SMD:R_0805_2012Metric" (layer "F.Cu")
+    (at 171.704 67.691 180)
+    (descr "Resistor SMD 0805 (2012 Metric), square (rectangular) end terminal, IPC_7351 nominal, (Body size source: IPC-SM-782 page 72, https://www.pcb-3d.com/wordpress/wp-content/uploads/ipc-sm-782a_amendment_1_and_2.pdf), generated with kicad-footprint-generator")
+    (tags "resistor")
+    (property "LCSC" "C17560")
+    (property "Sheetfile" "cut.kicad_sch")
+    (property "Sheetname" "DCC cutting")
+    (attr smd)
+    (fp_text reference "R34" (at 0 -1.65) (layer "F.SilkS")
+      (effects (font (size 1 1) (thickness 0.15)))
+    )
+    (fp_text value "22k" (at 0 1.65) (layer "F.Fab")
+      (effects (font (size 1 1) (thickness 0.15)))
+    )
+    (fp_text user "${REFERENCE}" (at 0 0) (layer "F.Fab")
+      (effects (font (size 0.5 0.5) (thickness 0.08)))
+    )
+    (fp_line (start -0.227064 -0.735) (end 0.227064 -0.735) (layer "F.SilkS") (width 0.12))
+    (fp_line (start -0.227064 0.735) (end 0.227064 0.735) (layer "F.SilkS") (width 0.12))
+    (fp_line (start -1.68 -0.95) (end 1.68 -0.95) (layer "F.CrtYd") (width 0.05))
+    (fp_line (start 1.68 0.95) (end -1.68 0.95) (layer "F.CrtYd") (width 0.05))
+    (fp_line (start -1.68 0.95) (end -1.68 -0.95) (layer "F.CrtYd") (width 0.05))
+    (fp_line (start 1.68 -0.95) (end 1.68 0.95) (layer "F.CrtYd") (width 0.05))
+    (fp_line (start -1 0.625) (end -1 -0.625) (layer "F.Fab") (width 0.1))
+    (fp_line (start -1 -0.625) (end 1 -0.625) (layer "F.Fab") (width 0.1))
+    (fp_line (start 1 -0.625) (end 1 0.625) (layer "F.Fab") (width 0.1))
+    (fp_line (start 1 0.625) (end -1 0.625) (layer "F.Fab") (width 0.1))
+    (pad "1" smd roundrect (at -0.9125 0 180) (size 1.025 1.4) (layers "F.Cu" "F.Paste" "F.Mask") (roundrect_rratio 0.243902)
+      (net 32 "Net-(D9-Pad2)") (pintype "passive"))
+    (pad "2" smd roundrect (at 0.9125 0 180) (size 1.025 1.4) (layers "F.Cu" "F.Paste" "F.Mask") (roundrect_rratio 0.243902)
+      (net 14 "Net-(C11-Pad2)") (pintype "passive"))
+    (model "${KICAD6_3DMODEL_DIR}/Resistor_SMD.3dshapes/R_0805_2012Metric.wrl"
+      (offset (xyz 0 0 0))
+      (scale (xyz 1 1 1))
+      (rotate (xyz 0 0 0))
+    )
+  )
+  (footprint "Resistor_SMD:R_0805_2012Metric" (layer "F.Cu")
     (at 128.016 89.154 180)
     (descr "Resistor SMD 0805 (2012 Metric), square (rectangular) end terminal, IPC_7351 nominal, (Body size source: IPC-SM-782 page 72, https://www.pcb-3d.com/wordpress/wp-content/uploads/ipc-sm-782a_amendment_1_and_2.pdf), generated with kicad-footprint-generator")
@@
     )
   )
+  (footprint "Resistor_SMD:R_0805_2012Metric" (layer "F.Cu")
+    (at 164.465 33.655)
+    (descr "Resistor SMD 0805 (2012 Metric), square (rectangular) end terminal, IPC_7351 nominal, (Body size source: IPC-SM-782 page 72, https://www.pcb-3d.com/wordpress/wp-content/uploads/ipc-sm-782a_amendment_1_and_2.pdf), generated with kicad-footprint-generator")
+    (tags "resistor")
+    (property "LCSC" "C17560")
+    (property "Sheetfile" "cut.kicad_sch")
+    (property "Sheetname" "DCC cutting")
+    (attr smd)
+    (fp_text reference "R33" (at 0 -1.65) (layer "F.SilkS")
+      (effects (font (size 1 1) (thickness 0.15)))
+    )
+    (fp_text value "22k" (at 0 1.65) (layer "F.Fab")
+      (effects (font (size 1 1) (thickness 0.15)))
+    )
+    (fp_text user "${REFERENCE}" (at 0 0) (layer "F.Fab")
+      (effects (font (size 0.5 0.5) (thickness 0.08)))
+    )
+    (fp_line (start -0.227064 0.735) (end 0.227064 0.735) (layer "F.SilkS") (width 0.12))
+    (fp_line (start -0.227064 -0.735) (end 0.227064 -0.735) (layer "F.SilkS") (width 0.12))
+    (fp_line (start -1.68 0.95) (end -1.68 -0.95) (layer "F.CrtYd") (width 0.05))
+    (fp_line (start 1.68 0.95) (end -1.68 0.95) (layer "F.CrtYd") (width 0.05))
+    (fp_line (start 1.68 -0.95) (end 1.68 0.95) (layer "F.CrtYd") (width 0.05))
+    (fp_line (start -1.68 -0.95) (end 1.68 -0.95) (layer "F.CrtYd") (width 0.05))
+    (fp_line (start -1 -0.625) (end 1 -0.625) (layer "F.Fab") (width 0.1))
+    (fp_line (start -1 0.625) (end -1 -0.625) (layer "F.Fab") (width 0.1))
+    (fp_line (start 1 -0.625) (end 1 0.625) (layer "F.Fab") (width 0.1))
+    (fp_line (start 1 0.625) (end -1 0.625) (layer "F.Fab") (width 0.1))
+    (pad "1" smd roundrect (at -0.9125 0) (size 1.025 1.4) (layers "F.Cu" "F.Paste" "F.Mask") (roundrect_rratio 0.243902)
+      (net 31 "Net-(D8-Pad2)") (pintype "passive"))
+    (pad "2" smd roundrect (at 0.9125 0) (size 1.025 1.4) (layers "F.Cu" "F.Paste" "F.Mask") (roundrect_rratio 0.243902)
+      (net 7 "Net-(C10-Pad1)") (pintype "passive"))
+    (model "${KICAD6_3DMODEL_DIR}/Resistor_SMD.3dshapes/R_0805_2012Metric.wrl"
+      (offset (xyz 0 0 0))
+      (scale (xyz 1 1 1))
+      (rotate (xyz 0 0 0))
+    )
+  )
   (footprint "Diode_SMD:D_SOD-123" (layer "F.Cu")
     (at 139.192 62.484)
@@
   (segment (start 122.682 114.7045) (end 122.682 124.0305) (width 0.3) (layer "F.Cu") (net 11))
   (segment (start 119.126 124.0305) (end 119.126 114.7045) (width 0.3) (layer "F.Cu") (net 12))
-  (segment (start 173.354 66.422) (end 173.354 65.278) (width 0.6) (layer "F.Cu") (net 13))
-  (segment (start 171.45 68.326) (end 173.354 66.422) (width 0.6) (layer "F.Cu") (net 13))
+  (segment (start 171.45 69.916) (end 170.241 69.916) (width 0.6) (layer "F.Cu") (net 13))
   (segment (start 173.354 65.278) (end 173.354 62.484) (width 0.6) (layer "F.Cu") (net 13))
   (segment (start 173.354 53.1355) (end 173.354 65.278) (width 0.3) (layer "F.Cu") (net 13))
+  (segment (start 170.241 69.916) (end 169.926 70.231) (width 0.6) (layer "F.Cu") (net 13))
   (segment (start 174.752 51.7375) (end 173.354 53.1355) (width 0.3) (layer "F.Cu") (net 13))
-  (segment (start 171.45 69.916) (end 171.45 68.326) (width 0.6) (layer "F.Cu") (net 13))
+  (segment (start 174.2065 69.916) (end 174.244 69.9535) (width 0.3) (layer "F.Cu") (net 13))
+  (segment (start 173.354 65.278) (end 171.704 65.278) (width 0.6) (layer "F.Cu") (net 13))
+  (segment (start 171.45 69.916) (end 174.2065 69.916) (width 0.3) (layer "F.Cu") (net 13))
+  (via (at 169.926 70.231) (size 1) (drill 0.6) (layers "F.Cu" "B.Cu") (net 13))
+  (via (at 171.704 65.278) (size 1) (drill 0.6) (layers "F.Cu" "B.Cu") (net 13))
+  (segment (start 171.704 68.453) (end 169.926 70.231) (width 0.6) (layer "In1.Cu") (net 13))
+  (segment (start 171.704 65.278) (end 171.704 68.326) (width 0.6) (layer "In1.Cu") (net 13))
+  (segment (start 171.704 68.326) (end 171.704 68.453) (width 0.6) (layer "In1.Cu") (net 13))
+  (segment (start 170.7915 67.691) (end 167.894 70.5885) (width 0.3) (layer "F.Cu") (net 14))
   (segment (start 167.894 69.342) (end 167.894 70.739) (width 0.6) (layer "F.Cu") (net 14))
   (segment (start 171.45 71.816) (end 168.971 71.816) (width 0.6) (layer "F.Cu") (net 14))
   (segment (start 164.466 65.278) (end 164.466 62.484) (width 0.6) (layer "F.Cu") (net 14))
+  (segment (start 167.894 70.5885) (end 167.894 70.739) (width 0.3) (layer "F.Cu") (net 14))
   (segment (start 164.466 65.278) (end 164.466 65.914) (width 0.6) (layer "F.Cu") (net 14))
   (segment (start 168.971 71.816) (end 167.894 70.739) (width 0.6) (layer "F.Cu") (net 14))
@@
   (segment (start 121.92 58.166) (end 121.92 57.15) (width 0.3) (layer "In1.Cu") (net 31))
   (segment (start 124.714 60.96) (end 121.92 58.166) (width 0.3) (layer "In1.Cu") (net 31))
-  (segment (start 174.244 69.9535) (end 174.244 68.326) (width 0.3) (layer "F.Cu") (net 32))
+  (segment (start 172.6165 67.691) (end 174.244 67.691) (width 0.3) (layer "F.Cu") (net 32))
   (segment (start 171.958 52.6565) (end 171.958 57.404) (width 0.3) (layer "F.Cu") (net 32))
   (segment (start 174.752 49.8625) (end 171.958 52.6565) (width 0.3) (layer "F.Cu") (net 32))
-  (via (at 174.244 68.326) (size 0.7) (drill 0.4) (layers "F.Cu" "B.Cu") (net 32))
+  (via (at 174.244 67.691) (size 0.7) (drill 0.4) (layers "F.Cu" "B.Cu") (net 32))
   (via (at 171.958 57.404) (size 0.8) (drill 0.4) (layers "F.Cu" "B.Cu") (net 32))
+  (segment (start 174.244 67.691) (end 174.244 59.69) (width 0.3) (layer "B.Cu") (net 32))
   (segment (start 174.244 59.69) (end 171.958 57.404) (width 0.3) (layer "B.Cu") (net 32))
-  (segment (start 174.244 68.326) (end 174.244 59.69) (width 0.3) (layer "B.Cu") (net 32))
   (segment (start 123.952 79.63) (end 123.952 75.702) (width 0.6) (layer "F.Cu") (net 33))
   (segment (start 127.753 80.255) (end 127.762 80.264) (width 0.6) (layer "F.Cu") (net 33))
