File: pcb/dc01.kicad_pcb (KiCad board)
At the start: 4 copper layers, 76 x 84 mm, 109 parts, among them J1 USB_C_Receptacle_USB2.0, J10 MV132, J2 PROG/DEBUG, J3 Conn_01x06, J4 RJ12, J5 RJ12, J6 MV132, J7 MV132, J8 Conn_01x02, J9 MV132, K1 AZ850-5, K2 AZ850-5, Q1 2N7002, Q2 2N7002, SW1 SW_Push, SW2 SW_Push, SW3 MFP 113 D, U1 STM32F103C8Tx, U2 AMS1117-3.3, U3 PC817, U4 PC817, U5 PC817, U6 PC817, U7 74HC123, Y1 8 MHz

Commit message: Tweak resistor values for LEDs.
Parts:
- moved R33 46.8 mm to (136.0, 70.9), turned to -90 degrees
- moved R10 12.1 mm to (148.7, 70.9)
Routing:
- net Net-(R10-Pad2): track 3.99 -> 11.6 mm
- net Net-(C10-Pad1): track 15.0 -> 22.6 mm
- net Net-(C10-Pad2): track 49.1 -> 51.5 mm
Changed lines of the file:
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@@
   )
   (footprint "Resistor_SMD:R_0805_2012Metric" (layer "F.Cu")
-    (at 136.652 70.866 -90)
+    (at 148.717 70.866 -90)
     (descr "Resistor SMD 0805 (2012 Metric), square (rectangular) end terminal, IPC_7351 nominal, (Body size source: IPC-SM-782 page 72, https://www.pcb-3d.com/wordpress/wp-content/uploads/ipc-sm-782a_amendment_1_and_2.pdf), generated with kicad-footprint-generator")
     (tags "resistor")
@@
     (property "Sheetname" "DCC cutting")
     (attr smd)
-    (fp_text reference "R10" (at 0 1.778 90) (layer "F.SilkS")
+    (fp_text reference "R10" (at -3.175 0 -90) (layer "F.SilkS")
       (effects (font (size 1 1) (thickness 0.15)))
     )
@@
     (property "Sheetname" "DCC cutting")
     (attr smd)
-    (fp_text reference "C10" (at 0 1.778 90) (layer "F.SilkS")
+    (fp_text reference "C10" (at -2.413 0 180) (layer "F.SilkS")
       (effects (font (size 1 1) (thickness 0.15)))
     )
@@
     (property "Sheetname" "DCC cutting")
     (attr smd)
-    (fp_text reference "R34" (at 0 -1.65) (layer "F.SilkS")
+    (fp_text reference "R34" (at 3.175 0 180) (layer "F.SilkS")
       (effects (font (size 1 1) (thickness 0.15)))
     )
@@
   )
   (footprint "Resistor_SMD:R_0805_2012Metric" (layer "F.Cu")
-    (at 164.465 33.655)
+    (at 136.017 70.866 -90)
     (descr "Resistor SMD 0805 (2012 Metric), square (rectangular) end terminal, IPC_7351 nominal, (Body size source: IPC-SM-782 page 72, https://www.pcb-3d.com/wordpress/wp-content/uploads/ipc-sm-782a_amendment_1_and_2.pdf), generated with kicad-footprint-generator")
     (tags "resistor")
@@
     (property "Sheetname" "DCC cutting")
     (attr smd)
-    (fp_text reference "R33" (at 0 -1.65) (layer "F.SilkS")
+    (fp_text reference "R33" (at 3.302 0 90) (layer "F.SilkS")
       (effects (font (size 1 1) (thickness 0.15)))
     )
-    (fp_text value "22k" (at 0 1.65) (layer "F.Fab")
+    (fp_text value "22k" (at 0 1.65 90) (layer "F.Fab")
       (effects (font (size 1 1) (thickness 0.15)))
     )
-    (fp_text user "${REFERENCE}" (at 0 0) (layer "F.Fab")
+    (fp_text user "${REFERENCE}" (at 0 0 90) (layer "F.Fab")
       (effects (font (size 0.5 0.5) (thickness 0.08)))
     )
@@
     (fp_line (start 1 -0.625) (end 1 0.625) (layer "F.Fab") (width 0.1))
     (fp_line (start 1 0.625) (end -1 0.625) (layer "F.Fab") (width 0.1))
-    (pad "1" smd roundrect (at -0.9125 0) (size 1.025 1.4) (layers "F.Cu" "F.Paste" "F.Mask") (roundrect_rratio 0.243902)
+    (pad "1" smd roundrect (at -0.9125 0 270) (size 1.025 1.4) (layers "F.Cu" "F.Paste" "F.Mask") (roundrect_rratio 0.243902)
       (net 31 "Net-(D8-Pad2)") (pintype "passive"))
-    (pad "2" smd roundrect (at 0.9125 0) (size 1.025 1.4) (layers "F.Cu" "F.Paste" "F.Mask") (roundrect_rratio 0.243902)
+    (pad "2" smd roundrect (at 0.9125 0 270) (size 1.025 1.4) (layers "F.Cu" "F.Paste" "F.Mask") (roundrect_rratio 0.243902)
       (net 7 "Net-(C10-Pad1)") (pintype "passive"))
     (model "${KICAD6_3DMODEL_DIR}/Resistor_SMD.3dshapes/R_0805_2012Metric.wrl"
@@
     (property "Sheetname" "DCC cutting")
     (attr smd)
-    (fp_text reference "D21" (at 0 2.032) (layer "F.SilkS")
+    (fp_text reference "D21" (at 3.302 0 90) (layer "F.SilkS")
       (effects (font (size 1 1) (thickness 0.15)))
     )
@@
     (property "Sheetname" "DCC cutting")
     (attr smd)
-    (fp_text reference "D22" (at 0 2.032) (layer "F.SilkS")
+    (fp_text reference "D22" (at -1.143 1.905) (layer "F.SilkS")
       (effects (font (size 1 1) (thickness 0.15)))
     )
@@
   (segment (start 151.139 82.305) (end 151.139 77.887) (width 0.6) (layer "In1.Cu") (net 6))
   (segment (start 159.258 110.028) (end 161.078 111.848) (width 0.6) (layer "In1.Cu") (net 6))
+  (segment (start 137.542 65.278) (end 137.542 70.992) (width 0.3) (layer "F.Cu") (net 7))
   (segment (start 143.825 71.816) (end 142.748 70.739) (width 0.6) (layer "F.Cu") (net 7))
   (segment (start 137.542 65.278) (end 137.542 62.484) (width 0.6) (layer "F.Cu") (net 7))
@@
   (segment (start 142.748 69.434) (end 142.748 70.739) (width 0.6) (layer "F.Cu") (net 7))
   (segment (start 137.542 65.278) (end 138.592 65.278) (width 0.6) (layer "F.Cu") (net 7))
+  (segment (start 136.7555 71.7785) (end 136.017 71.7785) (width 0.3) (layer "F.Cu") (net 7))
+  (segment (start 137.542 70.992) (end 136.7555 71.7785) (width 0.3) (layer "F.Cu") (net 7))
   (segment (start 146.43 67.944) (end 146.43 69.79) (width 0.6) (layer "F.Cu") (net 8))
+  (segment (start 148.717 69.9535) (end 146.3415 69.9535) (width 0.4) (layer "F.Cu") (net 8))
   (segment (start 121.92 49.8625) (end 121.92 48.006) (width 0.3) (layer "F.Cu") (net 8))
   (segment (start 146.43 65.278) (end 146.43 62.484) (width 0.6) (layer "F.Cu") (net 8))
@@
   (segment (start 147.828 67.818) (end 147.702 67.944) (width 0.3) (layer "F.Cu") (net 8))
   (segment (start 146.43 69.79) (end 146.304 69.916) (width 0.6) (layer "F.Cu") (net 8))
+  (segment (start 146.3415 69.9535) (end 146.304 69.916) (width 0.4) (layer "F.Cu") (net 8))
   (via (at 121.92 48.006) (size 0.8) (drill 0.4) (layers "F.Cu" "B.Cu") (net 8))
   (via (at 147.828 67.818) (size 0.8) (drill 0.4) (layers "F.Cu" "B.Cu") (net 8))
@@
   (segment (start 174.2065 69.916) (end 174.244 69.9535) (width 0.3) (layer "F.Cu") (net 13))
   (segment (start 173.354 65.278) (end 171.704 65.278) (width 0.6) (layer "F.Cu") (net 13))
-  (segment (start 171.45 69.916) (end 174.2065 69.916) (width 0.3) (layer "F.Cu") (net 13))
-  (via (at 169.926 70.231) (size 1) (drill 0.6) (layers "F.Cu" "B.Cu") (net 13))
-  (via (at 171.704 65.278) (size 1) (drill 0.6) (layers "F.Cu" "B.Cu") (net 13))
+  (segment (start 171.45 69.916) (end 174.2065 69.916) (width 0.4) (layer "F.Cu") (net 13))
+  (via (at 169.926 70.231) (size 0.8) (drill 0.4) (layers "F.Cu" "B.Cu") (net 13))
+  (via (at 171.704 65.278) (size 0.8) (drill 0.4) (layers "F.Cu" "B.Cu") (net 13))
   (segment (start 171.704 68.453) (end 169.926 70.231) (width 0.6) (layer "In1.Cu") (net 13))
   (segment (start 171.704 65.278) (end 171.704 68.326) (width 0.6) (layer "In1.Cu") (net 13))
@@
   (segment (start 137.562 57.298) (end 137.562 53.616) (width 0.6) (layer "F.Cu") (net 30))
   (segment (start 140.208 65.278) (end 139.192 64.262) (width 0.6) (layer "F.Cu") (net 30))
-  (segment (start 136.652 69.088) (end 135.382 67.818) (width 0.3) (layer "F.Cu") (net 31))
-  (segment (start 134.366 66.802) (end 134.366 62.484) (width 0.3) (layer "F.Cu") (net 31))
-  (segment (start 136.652 69.85) (end 136.652 69.088) (width 0.3) (layer "F.Cu") (net 31))
-  (segment (start 135.382 67.818) (end 134.366 66.802) (width 0.3) (layer "F.Cu") (net 31))
+  (segment (start 136.017 69.9535) (end 136.017 68.453) (width 0.3) (layer "F.Cu") (net 31))
   (segment (start 121.92 57.15) (end 121.92 51.7375) (width 0.3) (layer "F.Cu") (net 31))
   (segment (start 136.652 69.9535) (end 136.652 69.85) (width 0.3) (layer "F.Cu") (net 31))
+  (segment (start 134.366 66.802) (end 134.366 62.484) (width 0.3) (layer "F.Cu") (net 31))
+  (segment (start 136.017 68.453) (end 134.366 66.802) (width 0.3) (layer "F.Cu") (net 31))
   (via (at 134.366 62.484) (size 0.8) (drill 0.4) (layers "F.Cu" "B.Cu") (net 31))
   (via (at 121.92 57.15) (size 0.8) (drill 0.4) (layers "F.Cu" "B.Cu") (net 31))
@@
   (segment (start 173.99 78.0815) (end 171.196 78.0815) (width 0.3) (layer "F.Cu") (net 88))
   (segment (start 171.196 78.0815) (end 169.2675 78.0815) (width 0.3) (layer "F.Cu") (net 88))
-  (segment (start 136.652 71.7785) (end 139.1685 71.7785) (width 0.3) (layer "F.Cu") (net 89))
-  (segment (start 139.1685 71.7785) (end 140.208 70.739) (width 0.3) (layer "F.Cu") (net 89))
-  (segment (start 174.244 71.7785) (end 174.244 72.39) (width 0.3) (layer "F.Cu") (net 90))
-  (segment (start 174.244 72.39) (end 173.228 73.406) (width 0.3) (layer "F.Cu") (net 90))
-  (segment (start 173.228 73.406) (end 166.624 73.406) (width 0.3) (layer "F.Cu") (net 90))
+  (segment (start 148.209 73.152) (end 148.717 72.644) (width 0.4) (layer "F.Cu") (net 89))
+  (segment (start 140.843 73.152) (end 148.209 73.152) (width 0.4) (layer "F.Cu") (net 89))
+  (segment (start 148.717 72.644) (end 148.717 71.7785) (width 0.4) (layer "F.Cu") (net 89))
+  (segment (start 140.208 72.517) (end 140.843 73.152) (width 0.4) (layer "F.Cu") (net 89))
+  (segment (start 140.208 70.739) (end 140.208 72.517) (width 0.4) (layer "F.Cu") (net 89))
+  (segment (start 174.244 72.39) (end 173.482 73.152) (width 0.4) (layer "F.Cu") (net 90))
   (segment (start 165.354 72.136) (end 165.354 70.739) (width 0.3) (layer "F.Cu") (net 90))
-  (segment (start 166.624 73.406) (end 165.354 72.136) (width 0.3) (layer "F.Cu") (net 90))
+  (segment (start 174.244 71.7785) (end 174.244 72.39) (width 0.4) (layer "F.Cu") (net 90))
+  (segment (start 166.37 73.152) (end 165.354 72.136) (width 0.4) (layer "F.Cu") (net 90))
+  (segment (start 173.482 73.152) (end 166.37 73.152) (width 0.4) (layer "F.Cu") (net 90))
   (segment (start 126.3885 85.09) (end 126.3885 85.7485) (width 0.3) (layer "F.Cu") (net 91))
   (segment (start 129.1355 85.09) (end 126.3885 85.09) (width 0.3) (layer "F.Cu") (net 91))

Commit message: Move D12 & D13 to another position to keep isolation distance.
Parts:
- R14, R26, R7: value 1k -> 2k2
- R21, R3: value 1k -> 10k
- moved D12 78.4 mm to (117.6, 127.1), turned to -90 degrees
- moved D13 70.1 mm to (117.6, 122.9), turned to 90 degrees
- moved R26 51.4 mm to (116.3, 113.8), turned to -90 degrees
- moved R14 51.3 mm to (118.9, 113.8), turned to -90 degrees
- moved R7 2.54 mm to (121.7, 113.8)
- moved H1 2.11 mm to (102.1, 117.3)
- moved R6 2.03 mm to (124.7, 113.8)
- moved D4 1.78 mm to (120.9, 125.0)
- moved D3 1.52 mm to (124.2, 125.0)
- moved D7 1.52 mm to (108.5, 111.8)
- moved R1 1.52 mm to (112.0, 111.8)
- moved R2 1.52 mm to (105.2, 111.8)
- moved R5 1.52 mm to (127.8, 113.8)
- moved J1 1.35 mm to (108.2, 127.2)
- moved D2 1.27 mm to (127.5, 125.0)
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Routing:
- net GND: track 36.2 -> 9.59 mm
- net /DCC cutting/REL2CTRL: track 69.5 -> 71.8 mm
- net /LED_RED: track 26.3 -> 24.3 mm
- net USBD+: track 52.7 -> 54.1 mm
- net Net-(D12-Pad2): track 15.4 -> 14.0 mm
- net +5V: track 78.0 -> 79.2 mm
- net USBD-: track 52.8 -> 53.9 mm
- net /LED_BLUE: track 29.7 -> 28.6 mm
- net /DCC cutting/REL1CTRL: track 38.5 -> 37.5 mm
- net /SW_GO: track 24.4 -> 23.4 mm
- net /LED_YEL: track 23.2 -> 22.2 mm
