File: pcb/dc01.kicad_pcb (KiCad board)
At the start: 4 copper layers, 76 x 84 mm, 109 parts, among them J1 USB_C_Receptacle_USB2.0, J10 MV132, J2 PROG/DEBUG, J3 Conn_01x06, J4 RJ12, J5 RJ12, J6 MV132, J7 MV132, J8 Conn_01x02, J9 MV132, K1 AZ850-5, K2 AZ850-5, Q1 2N7002, Q2 2N7002, SW1 SW_Push, SW2 SW_Push, SW3 MFP 113 D, U1 STM32F103C8Tx, U2 AMS1117-3.3, U3 PC817, U4 PC817, U5 PC817, U6 PC817, U7 74HC123, Y1 8 MHz

Commit message: Increase DCC resistor value.
Other:
- board text added: "DC-01 v1.2"
- board text removed: "DC-01 v1.1"
Changed lines of the file:
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@@
     (effects (font (size 1.5 1.5) (thickness 0.15)))
   )
-  (gr_text "DC-01\nv1.1" (at 107.442 64.008) (layer "F.SilkS")
+  (gr_text "DC-01\nv1.2" (at 107.442 64.008) (layer "F.SilkS")
     (effects (font (size 2 2) (thickness 0.2)))
   )

Commit message: Use handsolder footprint for 1206 fuses.
Parts:
- F1, F2: footprint Fuse:Fuse_1206_3216Metric -> Fuse:Fuse_1206_3216Metric_Pad1.42x1.75mm_HandSolder
- R33, R34: value 22k -> 47k
Changed lines of the file:
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@@
     )
   )
-  (footprint "Fuse:Fuse_1206_3216Metric" (layer "F.Cu")
+  (footprint "Fuse:Fuse_1206_3216Metric_Pad1.42x1.75mm_HandSolder" (layer "F.Cu")
     (at 153.67 61.214 180)
-    (descr "Fuse SMD 1206 (3216 Metric), square (rectangular) end terminal, IPC_7351 nominal, (Body size source: http://www.tortai-tech.com/upload/download/2011102023233369053.pdf), generated with kicad-footprint-generator")
-    (tags "fuse")
+    (descr "Fuse SMD 1206 (3216 Metric), square (rectangular) end terminal, IPC_7351 nominal with elongated pad for handsoldering. (Body size source: http://www.tortai-tech.com/upload/download/2011102023233369053.pdf), generated with kicad-footprint-generator")
+    (tags "fuse handsolder")
     (property "JLCPCB_IGNORE" "true")
     (property "Sheetfile" "cut.kicad_sch")
     (property "Sheetname" "DCC cutting")
     (attr smd)
-    (fp_text reference "F1" (at 0 2.032) (layer "F.SilkS")
-      (effects (font (size 1 1) (thickness 0.15)))
-    )
-    (fp_text value "1A" (at 0 1.82) (layer "F.Fab")
-      (effects (font (size 1 1) (thickness 0.15)))
-    )
-    (fp_text user "${REFERENCE}" (at 0 0) (layer "F.Fab")
+    (fp_text reference "F1" (at 0 -1.82 180) (layer "F.SilkS")
+      (effects (font (size 1 1) (thickness 0.15)))
+    )
+    (fp_text value "1A" (at 0 1.82 180) (layer "F.Fab")
+      (effects (font (size 1 1) (thickness 0.15)))
+    )
+    (fp_text user "${REFERENCE}" (at 0 0 180) (layer "F.Fab")
       (effects (font (size 0.8 0.8) (thickness 0.12)))
     )
+    (fp_line (start -0.602064 0.91) (end 0.602064 0.91) (layer "F.SilkS") (width 0.12))
     (fp_line (start -0.602064 -0.91) (end 0.602064 -0.91) (layer "F.SilkS") (width 0.12))
-    (fp_line (start -0.602064 0.91) (end 0.602064 0.91) (layer "F.SilkS") (width 0.12))
-    (fp_line (start -2.28 -1.12) (end 2.28 -1.12) (layer "F.CrtYd") (width 0.05))
-    (fp_line (start -2.28 1.12) (end -2.28 -1.12) (layer "F.CrtYd") (width 0.05))
-    (fp_line (start 2.28 -1.12) (end 2.28 1.12) (layer "F.CrtYd") (width 0.05))
-    (fp_line (start 2.28 1.12) (end -2.28 1.12) (layer "F.CrtYd") (width 0.05))
+    (fp_line (start 2.45 1.12) (end -2.45 1.12) (layer "F.CrtYd") (width 0.05))
+    (fp_line (start 2.45 -1.12) (end 2.45 1.12) (layer "F.CrtYd") (width 0.05))
+    (fp_line (start -2.45 1.12) (end -2.45 -1.12) (layer "F.CrtYd") (width 0.05))
+    (fp_line (start -2.45 -1.12) (end 2.45 -1.12) (layer "F.CrtYd") (width 0.05))
+    (fp_line (start -1.6 -0.8) (end 1.6 -0.8) (layer "F.Fab") (width 0.1))
+    (fp_line (start -1.6 0.8) (end -1.6 -0.8) (layer "F.Fab") (width 0.1))
     (fp_line (start 1.6 -0.8) (end 1.6 0.8) (layer "F.Fab") (width 0.1))
     (fp_line (start 1.6 0.8) (end -1.6 0.8) (layer "F.Fab") (width 0.1))
-    (fp_line (start -1.6 -0.8) (end 1.6 -0.8) (layer "F.Fab") (width 0.1))
-    (fp_line (start -1.6 0.8) (end -1.6 -0.8) (layer "F.Fab") (width 0.1))
-    (pad "1" smd roundrect (at -1.4 0 180) (size 1.25 1.75) (layers "F.Cu" "F.Paste" "F.Mask") (roundrect_rratio 0.2)
+    (pad "1" smd roundrect (at -1.4875 0 180) (size 1.425 1.75) (layers "F.Cu" "F.Paste" "F.Mask") (roundrect_rratio 0.175439)
       (net 61 "Net-(D17-Pad1)") (pintype "passive"))
-    (pad "2" smd roundrect (at 1.4 0 180) (size 1.25 1.75) (layers "F.Cu" "F.Paste" "F.Mask") (roundrect_rratio 0.2)
+    (pad "2" smd roundrect (at 1.4875 0 180) (size 1.425 1.75) (layers "F.Cu" "F.Paste" "F.Mask") (roundrect_rratio 0.175439)
       (net 64 "/DCC cutting/J2") (pintype "passive"))
     (model "${KICAD6_3DMODEL_DIR}/Fuse.3dshapes/Fuse_1206_3216Metric.wrl"
@@
     (descr "Resistor SMD 0805 (2012 Metric), square (rectangular) end terminal, IPC_7351 nominal, (Body size source: IPC-SM-782 page 72, https://www.pcb-3d.com/wordpress/wp-content/uploads/ipc-sm-782a_amendment_1_and_2.pdf), generated with kicad-footprint-generator")
     (tags "resistor")
-    (property "LCSC" "C17560")
+    (property "LCSC" "C17713")
     (property "Sheetfile" "cut.kicad_sch")
     (property "Sheetname" "DCC cutting")
@@
       (effects (font (size 1 1) (thickness 0.15)))
     )
-    (fp_text value "22k" (at 0 1.65) (layer "F.Fab")
+    (fp_text value "47k" (at 0 1.65) (layer "F.Fab")
       (effects (font (size 1 1) (thickness 0.15)))
     )
@@
     (descr "Resistor SMD 0805 (2012 Metric), square (rectangular) end terminal, IPC_7351 nominal, (Body size source: IPC-SM-782 page 72, https://www.pcb-3d.com/wordpress/wp-content/uploads/ipc-sm-782a_amendment_1_and_2.pdf), generated with kicad-footprint-generator")
     (tags "resistor")
-    (property "LCSC" "C17560")
+    (property "LCSC" "C17713")
     (property "Sheetfile" "cut.kicad_sch")
     (property "Sheetname" "DCC cutting")
@@
       (effects (font (size 1 1) (thickness 0.15)))
     )
-    (fp_text value "22k" (at 0 1.65 90) (layer "F.Fab")
+    (fp_text value "47k" (at 0 1.65 90) (layer "F.Fab")
       (effects (font (size 1 1) (thickness 0.15)))
     )
@@
     )
   )
-  (footprint "Fuse:Fuse_1206_3216Metric" (layer "F.Cu")
+  (footprint "Fuse:Fuse_1206_3216Metric_Pad1.42x1.75mm_HandSolder" (layer "F.Cu")
     (at 159.766 61.214)
-    (descr "Fuse SMD 1206 (3216 Metric), square (rectangular) end terminal, IPC_7351 nominal, (Body size source: http://www.tortai-tech.com/upload/download/2011102023233369053.pdf), generated with kicad-footprint-generator")
-    (tags "fuse")
+    (descr "Fuse SMD 1206 (3216 Metric), square (rectangular) end terminal, IPC_7351 nominal with elongated pad for handsoldering. (Body size source: http://www.tortai-tech.com/upload/download/2011102023233369053.pdf), generated with kicad-footprint-generator")
+    (tags "fuse handsolder")
     (property "JLCPCB_IGNORE" "true")
     (property "Sheetfile" "cut.kicad_sch")
     (property "Sheetname" "DCC cutting")
     (attr smd)
-    (fp_text reference "F2" (at 0 -2.032) (layer "F.SilkS")
+    (fp_text reference "F2" (at 0 -1.82) (layer "F.SilkS")
       (effects (font (size 1 1) (thickness 0.15)))
     )
@@
     (fp_line (start -0.602064 0.91) (end 0.602064 0.91) (layer "F.SilkS") (width 0.12))
     (fp_line (start -0.602064 -0.91) (end 0.602064 -0.91) (layer "F.SilkS") (width 0.12))
-    (fp_line (start -2.28 1.12) (end -2.28 -1.12) (layer "F.CrtYd") (width 0.05))
-    (fp_line (start -2.28 -1.12) (end 2.28 -1.12) (layer "F.CrtYd") (width 0.05))
-    (fp_line (start 2.28 -1.12) (end 2.28 1.12) (layer "F.CrtYd") (width 0.05))
-    (fp_line (start 2.28 1.12) (end -2.28 1.12) (layer "F.CrtYd") (width 0.05))
+    (fp_line (start 2.45 1.12) (end -2.45 1.12) (layer "F.CrtYd") (width 0.05))
+    (fp_line (start -2.45 1.12) (end -2.45 -1.12) (layer "F.CrtYd") (width 0.05))
+    (fp_line (start -2.45 -1.12) (end 2.45 -1.12) (layer "F.CrtYd") (width 0.05))
+    (fp_line (start 2.45 -1.12) (end 2.45 1.12) (layer "F.CrtYd") (width 0.05))
+    (fp_line (start 1.6 0.8) (end -1.6 0.8) (layer "F.Fab") (width 0.1))
+    (fp_line (start 1.6 -0.8) (end 1.6 0.8) (layer "F.Fab") (width 0.1))
     (fp_line (start -1.6 -0.8) (end 1.6 -0.8) (layer "F.Fab") (width 0.1))
     (fp_line (start -1.6 0.8) (end -1.6 -0.8) (layer "F.Fab") (width 0.1))
-    (fp_line (start 1.6 0.8) (end -1.6 0.8) (layer "F.Fab") (width 0.1))
-    (fp_line (start 1.6 -0.8) (end 1.6 0.8) (layer "F.Fab") (width 0.1))
-    (pad "1" smd roundrect (at -1.4 0) (size 1.25 1.75) (layers "F.Cu" "F.Paste" "F.Mask") (roundrect_rratio 0.2)
+    (pad "1" smd roundrect (at -1.4875 0) (size 1.425 1.75) (layers "F.Cu" "F.Paste" "F.Mask") (roundrect_rratio 0.175439)
       (net 63 "Net-(D21-Pad1)") (pintype "passive"))
-    (pad "2" smd roundrect (at 1.4 0) (size 1.25 1.75) (layers "F.Cu" "F.Paste" "F.Mask") (roundrect_rratio 0.2)
+    (pad "2" smd roundrect (at 1.4875 0) (size 1.425 1.75) (layers "F.Cu" "F.Paste" "F.Mask") (roundrect_rratio 0.175439)
       (net 65 "/DCC cutting/K2") (pintype "passive"))
     (model "${KICAD6_3DMODEL_DIR}/Fuse.3dshapes/Fuse_1206_3216Metric.wrl"

Commit message: Switch active-alert outputs.
Connections:
- R23 pad 1: OUT_ALERT -> OUT_ON
- R24 pad 1: OUT_ON -> OUT_ALERT
Routing:
- net OUT_ON: track 49.2 -> 52.5 mm
- net OUT_ALERT: track 52.5 -> 49.2 mm
Changed lines of the file:
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@@
     (fp_line (start -1 -0.625) (end 1 -0.625) (layer "F.Fab") (width 0.1))
     (pad "1" smd roundrect (at -0.9125 0 90) (size 1.025 1.4) (layers "F.Cu" "F.Paste" "F.Mask") (roundrect_rratio 0.243902)
-      (net 99 "OUT_ON") (pintype "passive"))
+      (net 97 "OUT_ALERT") (pintype "passive"))
     (pad "2" smd roundrect (at 0.9125 0 90) (size 1.025 1.4) (layers "F.Cu" "F.Paste" "F.Mask") (roundrect_rratio 0.243902)
       (net 100 "Net-(R24-Pad2)") (pintype "passive"))
@@
     (fp_line (start -1 0.625) (end -1 -0.625) (layer "F.Fab") (width 0.1))
     (pad "1" smd roundrect (at -0.9125 0 90) (size 1.025 1.4) (layers "F.Cu" "F.Paste" "F.Mask") (roundrect_rratio 0.243902)
-      (net 97 "OUT_ALERT") (pintype "passive"))
+      (net 99 "OUT_ON") (pintype "passive"))
     (pad "2" smd roundrect (at 0.9125 0 90) (size 1.025 1.4) (layers "F.Cu" "F.Paste" "F.Mask") (roundrect_rratio 0.243902)
       (net 98 "Net-(R23-Pad2)") (pintype "passive"))
@@
   (segment (start 153.578 107.648) (end 151.478 105.548) (width 0.3) (layer "B.Cu") (net 96))
   (segment (start 151.478 105.548) (end 147.478 105.548) (width 0.3) (layer "B.Cu") (net 96))
-  (segment (start 144.1855 104.2555) (end 144.1855 107.5525) (width 0.3) (layer "F.Cu") (net 97))
-  (segment (start 104.9705 85.2405) (end 102.87 85.2405) (width 0.3) (layer "F.Cu") (net 97))
-  (segment (start 114.578 94.748) (end 114.478 94.748) (width 0.3) (layer "F.Cu") (net 97))
-  (segment (start 114.478 94.748) (end 104.9705 85.2405) (width 0.3) (layer "F.Cu") (net 97))
-  (via (at 114.578 94.748) (size 0.7) (drill 0.4) (layers "F.Cu" "B.Cu") (net 97))
-  (via (at 144.1855 104.2555) (size 0.7) (drill 0.4) (layers "F.Cu" "B.Cu") (net 97))
-  (segment (start 138.878 103.348) (end 123.178 103.348) (width 0.3) (layer "B.Cu") (net 97))
-  (segment (start 144.1855 104.2555) (end 139.7855 104.2555) (width 0.3) (layer "B.Cu") (net 97))
-  (segment (start 123.178 103.348) (end 114.578 94.748) (width 0.3) (layer "B.Cu") (net 97))
-  (segment (start 139.7855 104.2555) (end 138.878 103.348) (width 0.3) (layer "B.Cu") (net 97))
+  (segment (start 145.078 103.648) (end 145.078 106.248) (width 0.3) (layer "F.Cu") (net 97))
+  (segment (start 145.078 106.248) (end 144.6855 106.6405) (width 0.3) (layer "F.Cu") (net 97))
+  (segment (start 144.6855 106.6405) (end 144.6855 107.5525) (width 0.3) (layer "F.Cu") (net 97))
+  (segment (start 109.22 87.79) (end 109.22 85.2405) (width 0.3) (layer "F.Cu") (net 97))
+  (segment (start 145.178 103.548) (end 145.078 103.648) (width 0.3) (layer "F.Cu") (net 97))
+  (segment (start 116.178 94.748) (end 109.22 87.79) (width 0.3) (layer "F.Cu") (net 97))
+  (via (at 145.178 103.548) (size 0.7) (drill 0.4) (layers "F.Cu" "B.Cu") (net 97))
+  (via (at 116.178 94.748) (size 0.7) (drill 0.4) (layers "F.Cu" "B.Cu") (net 97))
+  (segment (start 144.48295 103.548) (end 144.47545 103.5555) (width 0.3) (layer "B.Cu") (net 97))
+  (segment (start 123.978 102.548) (end 116.178 94.748) (width 0.3) (layer "B.Cu") (net 97))
+  (segment (start 145.178 103.548) (end 144.48295 103.548) (width 0.3) (layer "B.Cu") (net 97))
+  (segment (start 138.978 102.548) (end 123.978 102.548) (width 0.3) (layer "B.Cu") (net 97))
+  (segment (start 144.47545 103.5555) (end 139.9855 103.5555) (width 0.3) (layer "B.Cu") (net 97))
+  (segment (start 139.9855 103.5555) (end 138.978 102.548) (width 0.3) (layer "B.Cu") (net 97))
   (segment (start 102.87 83.4155) (end 102.87 79.629) (width 0.3) (layer "F.Cu") (net 98))
-  (segment (start 145.078 103.648) (end 145.078 106.248) (width 0.3) (layer "F.Cu") (net 99))
-  (segment (start 145.078 106.248) (end 144.6855 106.6405) (width 0.3) (layer "F.Cu") (net 99))
-  (segment (start 144.6855 106.6405) (end 144.6855 107.5525) (width 0.3) (layer "F.Cu") (net 99))
-  (segment (start 109.22 87.79) (end 109.22 85.2405) (width 0.3) (layer "F.Cu") (net 99))
-  (segment (start 145.178 103.548) (end 145.078 103.648) (width 0.3) (layer "F.Cu") (net 99))
-  (segment (start 116.178 94.748) (end 109.22 87.79) (width 0.3) (layer "F.Cu") (net 99))
-  (via (at 145.178 103.548) (size 0.7) (drill 0.4) (layers "F.Cu" "B.Cu") (net 99))
-  (via (at 116.178 94.748) (size 0.7) (drill 0.4) (layers "F.Cu" "B.Cu") (net 99))
-  (segment (start 144.48295 103.548) (end 144.47545 103.5555) (width 0.3) (layer "B.Cu") (net 99))
-  (segment (start 123.978 102.548) (end 116.178 94.748) (width 0.3) (layer "B.Cu") (net 99))
-  (segment (start 145.178 103.548) (end 144.48295 103.548) (width 0.3) (layer "B.Cu") (net 99))
-  (segment (start 138.978 102.548) (end 123.978 102.548) (width 0.3) (layer "B.Cu") (net 99))
-  (segment (start 144.47545 103.5555) (end 139.9855 103.5555) (width 0.3) (layer "B.Cu") (net 99))
-  (segment (start 139.9855 103.5555) (end 138.978 102.548) (width 0.3) (layer "B.Cu") (net 99))
+  (segment (start 144.1855 104.2555) (end 144.1855 107.5525) (width 0.3) (layer "F.Cu") (net 99))
+  (segment (start 104.9705 85.2405) (end 102.87 85.2405) (width 0.3) (layer "F.Cu") (net 99))
+  (segment (start 114.578 94.748) (end 114.478 94.748) (width 0.3) (layer "F.Cu") (net 99))
+  (segment (start 114.478 94.748) (end 104.9705 85.2405) (width 0.3) (layer "F.Cu") (net 99))
+  (via (at 114.578 94.748) (size 0.7) (drill 0.4) (layers "F.Cu" "B.Cu") (net 99))
+  (via (at 144.1855 104.2555) (size 0.7) (drill 0.4) (layers "F.Cu" "B.Cu") (net 99))
+  (segment (start 138.878 103.348) (end 123.178 103.348) (width 0.3) (layer "B.Cu") (net 99))
+  (segment (start 144.1855 104.2555) (end 139.7855 104.2555) (width 0.3) (layer "B.Cu") (net 99))
+  (segment (start 123.178 103.348) (end 114.578 94.748) (width 0.3) (layer "B.Cu") (net 99))
+  (segment (start 139.7855 104.2555) (end 138.878 103.348) (width 0.3) (layer "B.Cu") (net 99))
   (segment (start 109.22 83.4155) (end 109.22 79.629) (width 0.3) (layer "F.Cu") (net 100))
   (segment (start 146.558 79.9065) (end 145.48 80.9845) (width 0.3) (layer "F.Cu") (net 101))
