File: pcb/cut.kicad_sch (KiCad schematic)
At the start: 34 parts, among them J4 RJ12, J5 RJ12, J6 Conn_01x02, J7 Conn_01x02, K1 AZ850-5, K2 AZ850-5, Q1 2N7002, Q2 2N7002, U5 PC817, U6 PC817

Commit message: Use dicrete schottky diodes for dcc rectifiers.
Schottky diodes do not cause short-time shortcuts.
Parts:
- removed D5, D6: D_Bridge_+-AA, Rectifiers:S250, symbol Device:D_Bridge_+-AA
- added D17, D18, D19, D20, D21, D22, D5, D6: 1N5819, Diode_SMD:D_SOD-123, symbol Diode:1N5819
Connections:
- net J1: now also D5.2 (A), D6.1 (K)
- net K1: now also D19.2 (A), D20.1 (K)
- net at C11.1, D9.1 (K): now also D17.2 (A), D21.2 (A)
- net at F1.1, K2.8: now also D17.1 (K), D18.2 (A)
- net at C10.1, U5.1: now also D19.1 (K), D5.1 (K)
- net at C10.2, D8.1 (K): now also D20.2 (A), D6.2 (A)
- net at F2.1, K2.3: now also D21.1 (K), D22.2 (A)
- net at C11.2, U6.1: now also D18.1 (K), D22.1 (K)
Other:
- moved on the sheet: C10, C11, D8, D9, R10, R11, R8, R9, U5, U6

Commit message: Add optocouplers output protection resistors.
Parts:
- added R29, R30: 1k, Resistor_SMD:R_0805_2012Metric, symbol Device:R
Connections:
- net IO1DCC: now also R29.1; no longer R8.1, U5.4
- net IO2DCC: now also R30.2; no longer R9.1, U6.4
- new net: R29.2, R8.1, U5.4
- new net: R30.1, R9.1, U6.4
Changed lines of the file:
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@@
   (junction (at 208.28 83.82) (diameter 0) (color 0 0 0 0)
   )
+  (junction (at 240.792 43.815) (diameter 0) (color 0 0 0 0)
+  )
+  (junction (at 125.73 98.425) (diameter 0) (color 0 0 0 0)
+  )
+  (junction (at 186.055 131.445) (diameter 0) (color 0 0 0 0)
+  )
+  (junction (at 40.64 102.87) (diameter 0) (color 0 0 0 0)
+  )
+  (junction (at 165.735 106.807) (diameter 0) (color 0 0 0 0)
+  )
+  (junction (at 105.41 106.68) (diameter 0) (color 0 0 0 0)
+  )
+  (junction (at 98.044 88.265) (diameter 0) (color 0 0 0 0)
+  )
+  (junction (at 52.197 43.815) (diameter 0) (color 0 0 0 0)
+  )
+  (junction (at 125.73 106.68) (diameter 0) (color 0 0 0 0)
+  )
   (junction (at 253.365 102.87) (diameter 0) (color 0 0 0 0)
   )
-  (junction (at 240.792 43.815) (diameter 0) (color 0 0 0 0)
-  )
-  (junction (at 125.73 98.425) (diameter 0) (color 0 0 0 0)
-  )
-  (junction (at 186.055 131.445) (diameter 0) (color 0 0 0 0)
-  )
-  (junction (at 165.735 106.807) (diameter 0) (color 0 0 0 0)
-  )
-  (junction (at 105.41 106.68) (diameter 0) (color 0 0 0 0)
-  )
-  (junction (at 98.044 88.265) (diameter 0) (color 0 0 0 0)
-  )
-  (junction (at 52.197 43.815) (diameter 0) (color 0 0 0 0)
-  )
-  (junction (at 125.73 106.68) (diameter 0) (color 0 0 0 0)
-  )
   (junction (at 208.28 95.25) (diameter 0) (color 0 0 0 0)
   )
   (junction (at 105.41 106.807) (diameter 0) (color 0 0 0 0)
-  )
-  (junction (at 40.64 102.87) (diameter 0) (color 0 0 0 0)
   )
   (junction (at 125.73 106.807) (diameter 0) (color 0 0 0 0)
@@
     (stroke (width 0) (type default) (color 0 0 0 0))
   )
+  (wire (pts (xy 253.365 102.87) (xy 260.985 102.87))
+    (stroke (width 0) (type default) (color 0 0 0 0))
+  )
   (wire (pts (xy 186.055 106.807) (xy 186.055 116.205))
     (stroke (width 0) (type default) (color 0 0 0 0))
@@
     (stroke (width 0) (type default) (color 0 0 0 0))
   )
+  (wire (pts (xy 22.86 102.87) (xy 26.67 102.87))
+    (stroke (width 0) (type default) (color 0 0 0 0))
+  )
   (wire (pts (xy 219.71 83.82) (xy 219.71 88.265))
     (stroke (width 0) (type default) (color 0 0 0 0))
@@
     (stroke (width 0) (type default) (color 0 0 0 0))
   )
-  (wire (pts (xy 253.365 102.87) (xy 263.525 102.87))
+  (wire (pts (xy 268.605 102.87) (xy 272.415 102.87))
     (stroke (width 0) (type default) (color 0 0 0 0))
   )
@@
     (stroke (width 0) (type default) (color 0 0 0 0))
   )
+  (wire (pts (xy 34.29 102.87) (xy 40.64 102.87))
+    (stroke (width 0) (type default) (color 0 0 0 0))
+  )
   (wire (pts (xy 253.365 107.95) (xy 253.365 111.125))
     (stroke (width 0) (type default) (color 0 0 0 0))
@@
   )
   (wire (pts (xy 183.515 98.425) (xy 186.055 98.425))
-    (stroke (width 0) (type default) (color 0 0 0 0))
-  )
-  (wire (pts (xy 40.64 102.87) (xy 30.48 102.87))
     (stroke (width 0) (type default) (color 0 0 0 0))
   )
@@
     (effects (font (size 1.27 1.27)) (justify left))
   )
-  (hierarchical_label "IO1DCC" (shape output) (at 30.48 102.87 180)
+  (hierarchical_label "IO1DCC" (shape output) (at 22.86 102.87 180)
     (effects (font (size 1.27 1.27)) (justify right))
   )
-  (hierarchical_label "IO2DCC" (shape output) (at 263.525 102.87 0)
+  (hierarchical_label "IO2DCC" (shape output) (at 272.415 102.87 0)
     (effects (font (size 1.27 1.27)) (justify left))
   )
@@
     (pin "2")
   )
+  (symbol (lib_id "Device:R") (at 30.48 102.87 90) (mirror x) (unit 1)
+    (in_bom yes) (on_board yes) (fields_autoplaced)
+    (property "Reference" "R29" (id 0) (at 30.48 98.1542 90))
+    (property "Value" "1k" (id 1) (at 30.48 100.6911 90))
+    (property "Footprint" "Resistor_SMD:R_0805_2012Metric" (id 2) (at 30.48 101.092 90)
+      (effects (font (size 1.27 1.27)) hide)
+    )
+    (property "Datasheet" "~" (id 3) (at 30.48 102.87 0)
+      (effects (font (size 1.27 1.27)) hide)
+    )
+    (property "LCSC" "C17414" (id 4) (at 30.48 102.87 0)
+      (effects (font (size 1.27 1.27)) hide)
+    )
+    (pin "1")
+    (pin "2")
+  )
   (symbol (lib_id "power:+5V") (at 165.735 96.52 0) (unit 1)
     (in_bom yes) (on_board yes)
@@
       (effects (font (size 1.27 1.27)) hide)
     )
+    (pin "1")
+    (pin "2")
+  )
+  (symbol (lib_id "Device:R") (at 264.795 102.87 90) (mirror x) (unit 1)
+    (in_bom yes) (on_board yes) (fields_autoplaced)
+    (property "Reference" "R30" (id 0) (at 264.795 98.1542 90))
+    (property "Value" "1k" (id 1) (at 264.795 100.6911 90))
+    (property "Footprint" "Resistor_SMD:R_0805_2012Metric" (id 2) (at 264.795 101.092 90)
+      (effects (font (size 1.27 1.27)) hide)
+    )
+    (property "Datasheet" "~" (id 3) (at 264.795 102.87 0)
+      (effects (font (size 1.27 1.27)) hide)
+    )
+    (property "LCSC" "C17414" (id 4) (at 264.795 102.87 0)
+      (effects (font (size 1.27 1.27)) hide)
+    )

Commit message: Use proper value for screw terminals.
Parts:
- J6, J7: value Conn_01x02 -> MVE252-5-V
Changed lines of the file:
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@@
     (in_bom yes) (on_board yes)
     (property "Reference" "J6" (id 0) (at 33.147 62.865 0))
-    (property "Value" "Conn_01x02" (id 1) (at 37.592 64.77 0))
+    (property "Value" "MVE252-5-V" (id 1) (at 37.592 64.77 0))
     (property "Footprint" "TerminalBlock_Euroclamp:MVE252-5-V" (id 2) (at 33.147 67.31 0)
       (effects (font (size 1.27 1.27)) hide)
@@
       (effects (font (size 1.27 1.27)) (justify left))
     )
-    (property "Value" "Conn_01x02" (id 1) (at 255.397 64.77 0))
+    (property "Value" "MVE252-5-V" (id 1) (at 255.397 64.77 0))
     (property "Footprint" "TerminalBlock_Euroclamp:MVE252-5-V" (id 2) (at 259.842 67.31 0)
       (effects (font (size 1.27 1.27)) hide)

Commit message: Use MV132 as screw terminals.
Parts:
- J6, J7: value MVE252-5-V -> MV132; footprint TerminalBlock_Euroclamp:MVE252-5-V -> TerminalBlock_4Ucon:TerminalBlock_4Ucon_1x02_P3.50mm_Horizontal
Changed lines of the file:
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@@
     (in_bom yes) (on_board yes)
     (property "Reference" "J6" (id 0) (at 33.147 62.865 0))
-    (property "Value" "MVE252-5-V" (id 1) (at 37.592 64.77 0))
-    (property "Footprint" "TerminalBlock_Euroclamp:MVE252-5-V" (id 2) (at 33.147 67.31 0)
+    (property "Value" "MV132" (id 1) (at 31.75 64.77 0)
+      (effects (font (size 1.27 1.27)) (justify right))
+    )
+    (property "Footprint" "TerminalBlock_4Ucon:TerminalBlock_4Ucon_1x02_P3.50mm_Horizontal" (id 2) (at 33.147 67.31 0)
       (effects (font (size 1.27 1.27)) hide)
     )
@@
       (effects (font (size 1.27 1.27)) (justify left))
     )
-    (property "Value" "MVE252-5-V" (id 1) (at 255.397 64.77 0))
-    (property "Footprint" "TerminalBlock_Euroclamp:MVE252-5-V" (id 2) (at 259.842 67.31 0)
+    (property "Value" "MV132" (id 1) (at 260.985 64.77 0)
+      (effects (font (size 1.27 1.27)) (justify right))
+    )
+    (property "Footprint" "TerminalBlock_4Ucon:TerminalBlock_4Ucon_1x02_P3.50mm_Horizontal" (id 2) (at 259.842 67.31 0)
       (effects (font (size 1.27 1.27)) hide)
     )

Commit message: Draw & route part of PCB.
Parts:
- D10, D11: footprint Diode_THT:D_DO-35_SOD27_P7.62mm_Horizontal -> Diode_SMD:D_0805_2012Metric_Pad1.15x1.40mm_HandSolder
Changed lines of the file:
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@@
     (property "Reference" "D11" (id 0) (at 175.895 109.855 0))
     (property "Value" "1N4148" (id 1) (at 175.895 111.76 0))
-    (property "Footprint" "Diode_THT:D_DO-35_SOD27_P7.62mm_Horizontal" (id 2) (at 175.895 111.125 0)
+    (property "Footprint" "Diode_SMD:D_0805_2012Metric_Pad1.15x1.40mm_HandSolder" (id 2) (at 175.895 111.125 0)
       (effects (font (size 1.27 1.27)) hide)
     )
@@
     (property "Reference" "D10" (id 0) (at 115.57 109.982 0))
     (property "Value" "1N4148" (id 1) (at 115.57 111.887 0))
-    (property "Footprint" "Diode_THT:D_DO-35_SOD27_P7.62mm_Horizontal" (id 2) (at 115.57 111.252 0)
+    (property "Footprint" "Diode_SMD:D_0805_2012Metric_Pad1.15x1.40mm_HandSolder" (id 2) (at 115.57 111.252 0)
       (effects (font (size 1.27 1.27)) hide)
     )
@@
   )
   (symbol (lib_id "Device:Polyfuse") (at 228.092 56.515 90) (unit 1)
-    (in_bom yes) (on_board yes) (fields_autoplaced)
-    (property "Reference" "F2" (id 0) (at 228.092 51.4182 90))
-    (property "Value" "1A" (id 1) (at 228.092 53.9551 90))
+    (in_bom yes) (on_board yes)
+    (property "Reference" "F2" (id 0) (at 227.965 60.96 90))
+    (property "Value" "1A" (id 1) (at 227.965 59.055 90))
     (property "Footprint" "Fuse:Fuse_1206_3216Metric" (id 2) (at 233.172 55.245 0)
       (effects (font (size 1.27 1.27)) (justify left) hide)

Commit message: Add LCSCs.
Parts:
- F1, F2, J6, J7, K1, K2: JLCPCB_IGNORE (none) -> true
- R10, R11: LCSC (none) -> C17520
- R29, R30: LCSC C17414 -> C17513
- U5, U6: LCSC (none) -> C106900
Changed lines of the file:
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@@
+      (effects (font (size 1.27 1.27)) hide)
+    )
+    (property "JLCPCB_IGNORE" "true" (id 4) (at 228.092 43.815 0)
       (effects (font (size 1.27 1.27)) hide)
     )
@@
       (effects (font (size 1.27 1.27)) (justify left) hide)
     )
+    (property "LCSC" "C106900" (id 4) (at 52.705 105.41 0)
+      (effects (font (size 1.27 1.27)) hide)
+    )
     (pin "1")
     (pin "2")
@@
       (effects (font (size 1.27 1.27)) hide)
     )
+    (property "JLCPCB_IGNORE" "true" (id 4) (at 228.092 56.515 0)
+      (effects (font (size 1.27 1.27)) hide)
+    )
     (pin "1")
     (pin "2")
@@
       (effects (font (size 1.27 1.27)) hide)
     )
+    (property "JLCPCB_IGNORE" "true" (id 4) (at 33.147 67.31 0)
+      (effects (font (size 1.27 1.27)) hide)
+    )
     (pin "1")
     (pin "2")
@@
     )
     (property "Datasheet" "http://www.azettler.com/pdfs/az850.pdf" (id 3) (at 175.895 88.265 0)
+      (effects (font (size 1.27 1.27)) hide)
+    )
+    (property "JLCPCB_IGNORE" "true" (id 4) (at 175.895 88.265 0)
       (effects (font (size 1.27 1.27)) hide)
     )
@@
       (effects (font (size 1.27 1.27)) hide)
     )
+    (property "JLCPCB_IGNORE" "true" (id 4) (at 259.842 67.31 0)
+      (effects (font (size 1.27 1.27)) hide)
+    )
     (pin "1")
     (pin "2")
@@
       (effects (font (size 1.27 1.27)) hide)
     )
-    (property "LCSC" "C17414" (id 4) (at 30.48 102.87 0)
+    (property "LCSC" "C17513" (id 4) (at 30.48 102.87 0)
       (effects (font (size 1.27 1.27)) hide)
     )
@@
       (effects (font (size 1.27 1.27)) hide)
     )
+    (property "LCSC" "C17520" (id 4) (at 73.66 107.95 0)
+      (effects (font (size 1.27 1.27)) hide)
+    )
     (pin "1")
     (pin "2")
@@
       (effects (font (size 1.27 1.27)) (justify left) hide)
     )
+    (property "LCSC" "C106900" (id 4) (at 241.3 105.41 0)
+      (effects (font (size 1.27 1.27)) hide)
+    )
     (pin "1")
     (pin "2")
@@
     )
     (property "Datasheet" "http://www.azettler.com/pdfs/az850.pdf" (id 3) (at 115.57 88.265 0)
+      (effects (font (size 1.27 1.27)) hide)
+    )
+    (property "JLCPCB_IGNORE" "true" (id 4) (at 115.57 88.265 0)
       (effects (font (size 1.27 1.27)) hide)
     )
@@
       (effects (font (size 1.27 1.27)) hide)
     )
+    (property "LCSC" "C17520" (id 4) (at 219.71 107.95 0)
+      (effects (font (size 1.27 1.27)) hide)
+    )
     (pin "1")
     (pin "2")
@@
       (effects (font (size 1.27 1.27)) hide)
     )
-    (property "LCSC" "C17414" (id 4) (at 264.795 102.87 0)
-      (effects (font (size 1.27 1.27)) hide)
-    )
+    (property "LCSC" "C17513" (id 4) (at 264.795 102.87 0)
+      (effects (font (size 1.27 1.27)) hide)
+    )

Commit message: Do not use 2 different types of diodes.
Parts:
- C12, C13: LCSC C45783 -> C15850
- D10, D11: value 1N4148 -> 1N5819; footprint Diode_SMD:D_0805_2012Metric_Pad1.15x1.40mm_HandSolder -> Diode_SMD:D_SOD-123; symbol Diode:1N4148 -> Diode:1N5819; LCSC C2128 -> C8598
Changed lines of the file:
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@@
     (pin "2")
   )
-  (symbol (lib_id "Diode:1N4148") (at 175.895 106.68 0) (unit 1)
+  (symbol (lib_id "Diode:1N5819") (at 175.895 106.68 0) (unit 1)
     (in_bom yes) (on_board yes)
     (property "Reference" "D11" (id 0) (at 175.895 109.855 0))
-    (property "Value" "1N4148" (id 1) (at 175.895 111.76 0))
-    (property "Footprint" "Diode_SMD:D_0805_2012Metric_Pad1.15x1.40mm_HandSolder" (id 2) (at 175.895 111.125 0)
-      (effects (font (size 1.27 1.27)) hide)
-    )
-    (property "Datasheet" "https://assets.nexperia.com/documents/data-sheet/1N4148_1N4448.pdf" (id 3) (at 175.895 106.68 0)
-      (effects (font (size 1.27 1.27)) hide)
-    )
-    (property "LCSC" "C2128" (id 4) (at 175.895 106.68 0)
+    (property "Value" "1N5819" (id 1) (at 175.895 111.76 0))
+    (property "Footprint" "Diode_SMD:D_SOD-123" (id 2) (at 175.895 111.125 0)
+      (effects (font (size 1.27 1.27)) hide)
+    )
+    (property "Datasheet" "http://www.vishay.com/docs/88525/1n5817.pdf" (id 3) (at 175.895 106.68 0)
+      (effects (font (size 1.27 1.27)) hide)
+    )
+    (property "LCSC" "C8598" (id 4) (at 175.895 106.68 0)
       (effects (font (size 1.27 1.27)) hide)
     )
@@
     (pin "2")
   )
-  (symbol (lib_id "Diode:1N4148") (at 115.57 106.807 0) (mirror y) (unit 1)
+  (symbol (lib_id "Diode:1N5819") (at 115.57 106.807 0) (mirror y) (unit 1)
     (in_bom yes) (on_board yes)
     (property "Reference" "D10" (id 0) (at 115.57 109.982 0))
-    (property "Value" "1N4148" (id 1) (at 115.57 111.887 0))
-    (property "Footprint" "Diode_SMD:D_0805_2012Metric_Pad1.15x1.40mm_HandSolder" (id 2) (at 115.57 111.252 0)
-      (effects (font (size 1.27 1.27)) hide)
-    )
-    (property "Datasheet" "https://assets.nexperia.com/documents/data-sheet/1N4148_1N4448.pdf" (id 3) (at 115.57 106.807 0)
-      (effects (font (size 1.27 1.27)) hide)
-    )
-    (property "LCSC" "C2128" (id 4) (at 115.57 106.807 0)
+    (property "Value" "1N5819" (id 1) (at 115.57 111.887 0))
+    (property "Footprint" "Diode_SMD:D_SOD-123" (id 2) (at 115.57 111.252 0)
+      (effects (font (size 1.27 1.27)) hide)
+    )
+    (property "Datasheet" "http://www.vishay.com/docs/88525/1n5817.pdf" (id 3) (at 115.57 106.807 0)
+      (effects (font (size 1.27 1.27)) hide)
+    )
+    (property "LCSC" "C8598" (id 4) (at 115.57 106.807 0)
       (effects (font (size 1.27 1.27)) hide)
     )
@@
       (effects (font (size 1.27 1.27)) hide)
     )
-    (property "LCSC" "C45783" (id 4) (at 125.73 116.205 0)
+    (property "LCSC" "C15850" (id 4) (at 125.73 116.205 0)
       (effects (font (size 1.27 1.27)) hide)
     )
@@
       (effects (font (size 1.27 1.27)) hide)
     )
-    (property "LCSC" "C45783" (id 4) (at 165.735 116.205 0)
-      (effects (font (size 1.27 1.27)) hide)
-    )
+    (property "LCSC" "C15850" (id 4) (at 165.735 116.205 0)
+      (effects (font (size 1.27 1.27)) hide)
+    )

Commit message: Conn → screw terminals.
Parts:
- J6, J7: symbol Connector_Generic:Conn_01x02 -> Connector:Screw_Terminal_01x02
Changed lines of the file:
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@@
     (pin "2")
   )
-  (symbol (lib_id "Connector_Generic:Conn_01x02") (at 33.147 67.31 0) (mirror y) (unit 1)
+  (symbol (lib_id "Connector:Screw_Terminal_01x02") (at 33.147 67.31 0) (mirror y) (unit 1)
     (in_bom yes) (on_board yes)
     (property "Reference" "J6" (id 0) (at 33.147 62.865 0))
@@
     (pin "1")
   )
-  (symbol (lib_id "Connector_Generic:Conn_01x02") (at 259.842 67.31 0) (unit 1)
+  (symbol (lib_id "Connector:Screw_Terminal_01x02") (at 259.842 67.31 0) (unit 1)
     (in_bom yes) (on_board yes)
     (property "Reference" "J7" (id 0) (at 258.572 62.865 0)
