File: pcb/cut.kicad_sch (KiCad schematic)
At the start: 42 parts, among them J4 RJ12, J5 RJ12, J6 MV132, J7 MV132, K1 AZ850-5, K2 AZ850-5, Q1 2N7002, Q2 2N7002, U5 PC817, U6 PC817

Commit message: Add separate resistors for LEDs.
Parts:
- added R33, R34: 22k, Resistor_SMD:R_0805_2012Metric, symbol Device:R
Connections:
- net at C11.1, D17.2 (A), D21.2 (A)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: now also R11.1
- net at D9.2 (A): now also R34.1; no longer R11.1
- net at C10.2, D20.2 (A), D6.2 (A)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: now also R10.1
- net at C10.1, D19.1 (K), D5.1 (K)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: now also R33.2
- net at D8.2 (A): now also R33.1; no longer R10.1
- net at C11.2, D18.1 (K), D22.1 (K)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: now also R34.2
Other:
- moved on the sheet: D12, D13, D8, D9, Q1, Q2, R10, R11, R12, R13, R14, R15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

Commit message: Tweak resistor values for LEDs.
Parts:
- R14, R26: value 1k -> 2k2; LCSC C17513 -> C17520
Changed lines of the file:
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@@
       (effects (font (size 1.27 1.27)) (justify left))
     )
-    (property "Value" "1k" (id 1) (at 212.979 134.4172 0)
+    (property "Value" "2k2" (id 1) (at 212.979 134.4172 0)
       (effects (font (size 1.27 1.27)) (justify left))
     )
@@
       (effects (font (size 1.27 1.27)) hide)
     )
-    (property "LCSC" "C17513" (id 4) (at 211.201 132.715 0)
+    (property "LCSC" "C17520" (id 4) (at 211.201 132.715 0)
       (effects (font (size 1.27 1.27)) hide)
     )
@@
   )
   (symbol (lib_id "Device:R") (at 80.645 132.715 0) (mirror y) (unit 1)
-    (in_bom yes) (on_board yes) (fields_autoplaced)
-    (property "Reference" "R14" (id 0) (at 78.867 131.8803 0)
-      (effects (font (size 1.27 1.27)) (justify left))
-    )
-    (property "Value" "1k" (id 1) (at 78.867 134.4172 0)
+    (in_bom yes) (on_board yes)
+    (property "Reference" "R14" (id 0) (at 78.74 132.08 0)
+      (effects (font (size 1.27 1.27)) (justify left))
+    )
+    (property "Value" "2k2" (id 1) (at 78.74 134.62 0)
       (effects (font (size 1.27 1.27)) (justify left))
     )
@@
       (effects (font (size 1.27 1.27)) hide)
     )
-    (property "LCSC" "C17513" (id 4) (at 80.645 132.715 0)
-      (effects (font (size 1.27 1.27)) hide)
-    )
+    (property "LCSC" "C17520" (id 4) (at 80.645 132.715 0)
+      (effects (font (size 1.27 1.27)) hide)
+    )

Commit message: Increase DCC resistor value.
Parts:
- R33, R34: value 22k -> 47k; LCSC C17560 -> C17713
Changed lines of the file:
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@@
     (in_bom yes) (on_board yes)
     (property "Reference" "R33" (id 0) (at 68.58 107.95 90))
-    (property "Value" "22k" (id 1) (at 68.58 103.2311 90))
+    (property "Value" "47k" (id 1) (at 68.58 103.2311 90))
     (property "Footprint" "Resistor_SMD:R_0805_2012Metric" (id 2) (at 68.58 107.188 90)
       (effects (font (size 1.27 1.27)) hide)
@@
       (effects (font (size 1.27 1.27)) hide)
     )
-    (property "LCSC" "C17560" (id 4) (at 68.58 105.41 0)
+    (property "LCSC" "C17713" (id 4) (at 68.58 105.41 0)
       (effects (font (size 1.27 1.27)) hide)
     )
@@
     (in_bom yes) (on_board yes)
     (property "Reference" "R34" (id 0) (at 224.155 107.95 90))
-    (property "Value" "22k" (id 1) (at 224.155 103.2311 90))
+    (property "Value" "47k" (id 1) (at 224.155 103.2311 90))
     (property "Footprint" "Resistor_SMD:R_0805_2012Metric" (id 2) (at 224.155 107.188 90)
       (effects (font (size 1.27 1.27)) hide)
@@
       (effects (font (size 1.27 1.27)) hide)
     )
-    (property "LCSC" "C17560" (id 4) (at 224.155 105.41 0)
-      (effects (font (size 1.27 1.27)) hide)
-    )
+    (property "LCSC" "C17713" (id 4) (at 224.155 105.41 0)
+      (effects (font (size 1.27 1.27)) hide)
+    )

Commit message: Use handsolder footprint for 1206 fuses.
Parts:
- F1, F2: footprint Fuse:Fuse_1206_3216Metric -> Fuse:Fuse_1206_3216Metric_Pad1.42x1.75mm_HandSolder
Changed lines of the file:
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@@
     (property "Reference" "F1" (id 0) (at 228.092 38.7182 90))
     (property "Value" "1A" (id 1) (at 228.092 41.2551 90))
-    (property "Footprint" "Fuse:Fuse_1206_3216Metric" (id 2) (at 233.172 42.545 0)
+    (property "Footprint" "Fuse:Fuse_1206_3216Metric_Pad1.42x1.75mm_HandSolder" (id 2) (at 233.172 42.545 0)
       (effects (font (size 1.27 1.27)) (justify left) hide)
     )
@@
     (property "Reference" "F2" (id 0) (at 227.965 60.96 90))
     (property "Value" "1A" (id 1) (at 227.965 59.055 90))
-    (property "Footprint" "Fuse:Fuse_1206_3216Metric" (id 2) (at 233.172 55.245 0)
+    (property "Footprint" "Fuse:Fuse_1206_3216Metric_Pad1.42x1.75mm_HandSolder" (id 2) (at 233.172 55.245 0)
       (effects (font (size 1.27 1.27)) (justify left) hide)
     )
